Commit message: Add complete gazebo launch with manipulator on the floor

File: aerial_manipulators_description/urdf/wp_manipulator.base.urdf.xacro (robot description, xacro)
@@ -5,5 +5,5 @@
   <xacro:wp_manipulator
     parent="world">
-    <origin xyz="0 0 0.5" rpy="${pi/2} 0 ${pi}"/>
+    <origin xyz="0 0 0.035" rpy="${pi/2} 0 ${pi}"/>
   </xacro:wp_manipulator>
    <xacro:transmisija
