Commit message: implemented direct kinematics for wp manipulator

File: aerial_manipulators_description/urdf/manipulator_base.urdf.xacro (robot description, xacro)
@@ -17,7 +17,7 @@
     <xacro:property name="mass5" value="${mass2*d5/a2}"/>
     <xacro:property name="rad" value="0.03"/>
-    <link name='link0'>
+    <link name='base'>
       <visual>
-        <origin xyz="0 0 0" rpy="${pi / 2} 0 ${pi}" />
+        <origin xyz="0 0 0" rpy="0 0 0" />
         <geometry>
           <mesh filename="package://aerial_manipulators_description/meshes/wp_manipulator/base.dae"
@@ -111,15 +111,10 @@
       </visual>
     </link>
-    <!--joint name="world_to_link0" type="fixed">
-      <parent link="world"/>
-      <child link="link0"/-->
-      <!-- Adjust Gazebo coordinate system to link1 coordinate system -->
-      <!--origin xyz="0 0 ${a0}" rpy="0 0 0"/>
-    </joint-->
+    <link name='end_effector_base'/>
     <joint name="joint1" type="revolute">
-      <parent link="link0"/>
+      <parent link="base"/>
       <child link="link1"/>
       <!-- Adjust Gazebo coordinate system to link1 coordinate system -->
-      <origin xyz="0 0 0" rpy="${pi/2} 0 ${pi}"/>
+      <origin xyz="0 0 0" rpy="0 0 0"/>
       <limit upper="1.57" lower="-1.57" effort="10000000" velocity="46"/>
       <axis xyz="0 0 1" />
@@ -129,6 +124,6 @@
       <child link="link2"/>
       <origin xyz="0 ${a1} 0" rpy="0 0 ${theta1}"/>
-      <limit upper="2.2" lower="-2.2" effort="10000000" velocity="46"/>
-      <axis xyz="0 0 -1" />
+      <limit upper="2.0" lower="-2.0" effort="10000000" velocity="46"/>
+      <axis xyz="0 0 1" />
     </joint>
     <joint name="joint3" type="revolute">
@@ -137,5 +132,5 @@
       <origin xyz="${a2} 0 0" rpy="${alpha2} 0 0"/>
       <limit upper="1.57" lower="-1.57" effort="10000000" velocity="46"/>
-      <axis xyz="0 0 -1" />
+      <axis xyz="0 0 1" />
     </joint>
     <joint name="joint4" type="revolute">
@@ -146,5 +141,4 @@
       <axis xyz="0 0 1" />
     </joint>
-<!-- <limit upper="1.57" lower="-1.57" effort="10000000" velocity="20"/> -->
     <joint name="joint5" type="revolute">
       <parent link="link4"/>
@@ -152,7 +146,11 @@
       <origin xyz="${a4} 0 0" rpy="0 0 0"/>
       <limit upper="2.3" lower="-2.3" effort="10000000" velocity="46"/>
-      <axis xyz="0 0 -1" />
+      <axis xyz="0 0 1" />
     </joint>
-<!--       <limit upper="2.3" lower="-2.3" effort="10000000" velocity="20"/> -->
+    <joint name="jointEndEffectorBase" type="fixed">
+      <parent link="link5"/>
+      <child link="end_effector_base"/>
+      <origin xyz="${d5} 0 0" rpy="0 0 0"/>
+    </joint>
   </xacro:macro>
   <!-- We add a <transmission> block for every joint that we wish to actuate. -->

File: aerial_manipulators_description/urdf/wp_manipulator.base.urdf.xacro (robot description, xacro)
@@ -6,30 +6,3 @@
     <origin xyz="0 0 0" rpy="0 0 0"/>
   </xacro:wp_manipulator>
-  <link name='world'/>
-  <joint name="world_to_link0" type="fixed">
-      <parent link="world"/>
-      <child link="link0"/>
-      <!-- Adjust Gazebo coordinate system to link1 coordinate system -->
-      <!--origin xyz="0 0 ${a0}" rpy="0 0 0"/-->
-    </joint>
-  <xacro:transmisija
-    trans_number="1"
-    joint_name="joint1">
-  </xacro:transmisija>
-  <xacro:transmisija
-    trans_number="2"
-    joint_name="joint2">
-  </xacro:transmisija>
-  <xacro:transmisija
-    trans_number="3"
-    joint_name="joint3">
-  </xacro:transmisija>
-  <xacro:transmisija
-    trans_number="4"
-    joint_name="joint4">
-  </xacro:transmisija>
-  <xacro:transmisija
-    trans_number="5"
-    joint_name="joint5">
-  </xacro:transmisija>
 </robot>

Commit message: working ik

File: aerial_manipulators_description/urdf/manipulator_base.urdf.xacro (robot description, xacro)
@@ -138,5 +138,5 @@
       <child link="link4"/>
       <origin xyz="${a3} 0 0" rpy="0 0 0"/>
-      <limit upper="1.57" lower="-1.57" effort="10000000" velocity="46"/>
+      <limit upper="2.0" lower="-2.0" effort="10000000" velocity="46"/>
       <axis xyz="0 0 1" />
     </joint>

Commit message: added new fixed joint in wp manipulator

File: aerial_manipulators_description/urdf/manipulator_base.urdf.xacro (robot description, xacro)
@@ -112,4 +112,9 @@
     </link>
     <link name='end_effector_base'/>
+    <joint name="base_joint" type="fixed">
+      <parent link="${parent}"/>
+      <child link="base"/>
+      <xacro:insert_block name="origin"/>
+    </joint>
     <joint name="joint1" type="revolute">
       <parent link="base"/>

File: aerial_manipulators_description/urdf/wp_manipulator.base.urdf.xacro (robot description, xacro)
@@ -2,4 +2,5 @@
 <robot name="wp_manipulator" xmlns:xacro="http://ros.org/wiki/xacro">
   <xacro:include filename="$(find aerial_manipulators_description)/urdf/manipulator_base.urdf.xacro" />
+  <link name="world"></link>
   <xacro:wp_manipulator
     parent="world">

Commit message: example of spawning wp manipulator

File: aerial_manipulators_description/urdf/manipulator_base.urdf.xacro (robot description, xacro)
@@ -18,4 +18,12 @@
     <xacro:property name="rad" value="0.03"/>
     <link name='base'>
+      <inertial>
+        <mass value="${mass5}" />
+        <origin xyz="0 -${d5/2} 0" rpy="0 0 0"/>
+        <inertia
+          ixx="${1/2 * mass5 * rad * rad}" ixy="0" ixz="0"
+          iyx="0" iyy="${1/12 * mass5 * (3*rad*rad + d5*d5)}" iyz="0"
+          izx="0" izy="0" izz="${1/12 * mass5 * (3*rad*rad + d5*d5)}"/>
+      </inertial>
       <visual>
         <origin xyz="0 0 0" rpy="0 0 0" />

Commit message: Add transmissions, mass and manipulator namespace.

File: aerial_manipulators_description/urdf/manipulator_base.urdf.xacro (robot description, xacro)
@@ -119,5 +119,19 @@
       </visual>
     </link>
-    <link name='end_effector_base'/>
+    <link name='end_effector_base'>
+      <inertial>
+        <mass value="0.00001" />
+        <origin xyz="0 0 0" rpy="0 0 0"/>
+        <inertia
+          ixx="0.00001" ixy="0" ixz="0"
+          iyx="0" iyy="0.00001" iyz="0"
+          izx="0" izy="0" izz="0.00001"/>
+      </inertial>
+      <visual>
+        <geometry>
+          <sphere radius="0.005"/>
+        </geometry>
+      </visual>
+    </link>
     <joint name="base_joint" type="fixed">
       <parent link="${parent}"/>

File: aerial_manipulators_description/urdf/wp_manipulator.base.urdf.xacro (robot description, xacro)
@@ -5,5 +5,25 @@
   <xacro:wp_manipulator
     parent="world">
-    <origin xyz="0 0 0" rpy="0 0 0"/>
+    <origin xyz="0 0 0.5" rpy="${pi/2} 0 ${pi}"/>
   </xacro:wp_manipulator>
+   <xacro:transmisija
+    trans_number="1"
+    joint_name="joint1">
+  </xacro:transmisija>
+  <xacro:transmisija
+    trans_number="2"
+    joint_name="joint2">
+  </xacro:transmisija>
+  <xacro:transmisija
+    trans_number="3"
+    joint_name="joint3">
+  </xacro:transmisija>
+  <xacro:transmisija
+    trans_number="4"
+    joint_name="joint4">
+  </xacro:transmisija>
+  <xacro:transmisija
+    trans_number="5"
+    joint_name="joint5">
+  </xacro:transmisija>
 </robot>

Commit message: Rename base_joint to wp_base_joint

File: aerial_manipulators_description/urdf/manipulator_base.urdf.xacro (robot description, xacro)
@@ -134,5 +134,5 @@
       </visual>
     </link>
-    <joint name="base_joint" type="fixed">
+    <joint name="wp_base_joint" type="fixed">
       <parent link="${parent}"/>
       <child link="base"/>

Commit message: added new manipulator

File: aerial_manipulators_description/urdf/manipulator_base.urdf.xacro (robot description, xacro)
@@ -20,9 +20,9 @@
       <inertial>
         <mass value="${mass5}" />
-        <origin xyz="0 -${d5/2} 0" rpy="0 0 0"/>
+        <origin xyz="0 -${a0/2} 0" rpy="0 0 0"/>
         <inertia
           ixx="${1/2 * mass5 * rad * rad}" ixy="0" ixz="0"
-          iyx="0" iyy="${1/12 * mass5 * (3*rad*rad + d5*d5)}" iyz="0"
-          izx="0" izy="0" izz="${1/12 * mass5 * (3*rad*rad + d5*d5)}"/>
+          iyx="0" iyy="${1/12 * mass5 * (3*rad*rad + a0*a0)}" iyz="0"
+          izx="0" izy="0" izz="${1/12 * mass5 * (3*rad*rad + a0*a0)}"/>
       </inertial>
       <visual>
@@ -177,4 +177,136 @@
     <joint name="jointEndEffectorBase" type="fixed">
       <parent link="link5"/>
+      <child link="end_effector_base"/>
+      <origin xyz="${d5} 0 0" rpy="0 0 0"/>
+    </joint>
+  </xacro:macro>
+  <xacro:macro name="wp_manipulator_3R"
+  params="parent *origin">
+    <xacro:property name="a0" value="0.04526"/>
+    <xacro:property name="a1" value="0.122490"/>
+    <xacro:property name="a2" value="0.1365"/>
+    <xacro:property name="a3" value="0.075511"/>
+    <xacro:property name="a4" value="0.072489"/>
+    <xacro:property name="d5" value="0.04526"/>
+    <xacro:property name="theta1" value="${pi/2}"/>
+    <xacro:property name="alpha2" value="${-pi/2}"/>
+    <xacro:property name="mass2" value="0.03"/>
+    <xacro:property name="mass1" value="${mass2*a1/a2}"/>
+    <xacro:property name="mass3" value="${mass2*a3/a2}"/>
+    <xacro:property name="mass4" value="${mass2*a4/a2}"/>
+    <xacro:property name="mass5" value="${mass2*d5/a2}"/>
+    <xacro:property name="rad" value="0.03"/>
+    <link name='base'>
+      <inertial>
+        <mass value="${mass5}" />
+        <origin xyz="0 -${a0/2} 0" rpy="0 0 0"/>
+        <inertia
+          ixx="${1/2 * mass5 * rad * rad}" ixy="0" ixz="0"
+          iyx="0" iyy="${1/12 * mass5 * (3*rad*rad + a0*a0)}" iyz="0"
+          izx="0" izy="0" izz="${1/12 * mass5 * (3*rad*rad + a0*a0)}"/>
+      </inertial>
+      <visual>
+        <origin xyz="0 0 0" rpy="0 0 0" />
+        <geometry>
+          <mesh filename="package://aerial_manipulators_description/meshes/wp_manipulator/base.dae"
+            scale="1 1 1" />
+        </geometry>
+      </visual>
+    </link>
+    <link name='link1'>
+      <inertial>
+        <mass value="${mass2}" />
+        <origin xyz="${a2/2} 0 0" rpy="0 0 0"/>
+        <inertia
+          ixx="${1/2 * mass2 * rad * rad}" ixy="0" ixz="0"
+          iyx="0" iyy="${1/12 * mass2 * (3*rad*rad + a2*a2)}" iyz="0"
+          izx="0" izy="0" izz="${1/12 * mass2 * (3*rad*rad + a2*a2)}"/>
+      </inertial>
+      <visual>
+        <origin xyz="0 0 0" rpy="0 0 0" />
+        <geometry>
+          <mesh filename="package://aerial_manipulators_description/meshes/wp_manipulator/link2_rotated.dae"
+            scale="1 1 1" />
+        </geometry>
+      </visual>
+    </link>
+    <link name='link2'>
+      <inertial>
+        <mass value="${mass4}" />
+        <origin xyz="${a4/2} 0 0" rpy="0 0 0"/>
+        <inertia
+          ixx="${1/2 * mass4 * rad * rad}" ixy="0" ixz="0"
+          iyx="0" iyy="${1/12 * mass4 * (3*rad*rad + a4*a4)}" iyz="0"
+          izx="0" izy="0" izz="${1/12 * mass4 * (3*rad*rad + a4*a4)}"/>
+      </inertial>
+      <visual>
+        <origin xyz="0 0 0" rpy="0 ${pi/2} ${-pi/2}" />
+        <geometry>
+          <mesh filename="package://aerial_manipulators_description/meshes/wp_manipulator/link4.dae"
+            scale="1 1 1" />
+        </geometry>
+      </visual>
+    </link>
+    <link name='link3'>
+      <inertial>
+        <mass value="${mass5}" />
+        <origin xyz="${a0/2} 0 0" rpy="0 0 0"/>
+        <inertia
+          ixx="${1/2 * mass5 * rad * rad}" ixy="0" ixz="0"
+          iyx="0" iyy="${1/12 * mass5 * (3*rad*rad + a0*a0)}" iyz="0"
+          izx="0" izy="0" izz="${1/12 * mass5 * (3*rad*rad + a0*a0)}"/>
+      </inertial>
+      <visual>
+        <origin xyz="0 0 0" rpy="0 ${pi / 2} 0" />
+        <geometry>
+          <mesh filename="package://aerial_manipulators_description/meshes/wp_manipulator/link5.dae"
+            scale="1 1 1" />
+        </geometry>
+      </visual>
+    </link>
+    <link name='end_effector_base'>
+      <inertial>
+        <mass value="0.00001" />
+        <origin xyz="0 0 0" rpy="0 0 0"/>
+        <inertia
+          ixx="0.00001" ixy="0" ixz="0"
+          iyx="0" iyy="0.00001" iyz="0"
+          izx="0" izy="0" izz="0.00001"/>
+      </inertial>
+      <visual>
+        <geometry>
+          <sphere radius="0.005"/>
+        </geometry>
+      </visual>
+    </link>
+    <joint name="wp_base_joint" type="fixed">
+      <parent link="${parent}"/>
+      <child link="base"/>
+      <xacro:insert_block name="origin"/>
+    </joint>
+    <joint name="joint1" type="revolute">
+      <parent link="base"/>
+      <child link="link1"/>
+      <!-- Adjust Gazebo coordinate system to link1 coordinate system -->
+      <origin xyz="0 0 0" rpy="0 0 0"/>
+      <limit upper="1.57" lower="-1.57" effort="10000000" velocity="46"/>
+      <axis xyz="0 0 1" />
+    </joint>
+    <joint name="joint2" type="revolute">
+      <parent link="link1"/>
+      <child link="link2"/>
+      <origin xyz="0 ${a2} 0" rpy="${-pi/2} 0 ${pi/2}"/>
+      <limit upper="2.0" lower="-2.0" effort="10000000" velocity="46"/>
+      <axis xyz="0 0 1" />
+    </joint>
+    <joint name="joint3" type="revolute">
+      <parent link="link2"/>
+      <child link="link3"/>
+      <origin xyz="${a4} 0 0" rpy="0 0 0"/>
+      <limit upper="2.3" lower="-2.3" effort="10000000" velocity="46"/>
+      <axis xyz="0 0 1" />
+    </joint>
+    <joint name="jointEndEffectorBase" type="fixed">
+      <parent link="link3"/>
       <child link="end_effector_base"/>
       <origin xyz="${d5} 0 0" rpy="0 0 0"/>

Commit message: fixed robot names

File: aerial_manipulators_description/urdf/manipulator_base.urdf.xacro (robot description, xacro)
@@ -188,5 +188,5 @@
     <xacro:property name="a3" value="0.075511"/>
     <xacro:property name="a4" value="0.072489"/>
-    <xacro:property name="d5" value="0.04526"/>
+    <xacro:property name="d5" value="0.035"/>
     <xacro:property name="theta1" value="${pi/2}"/>
     <xacro:property name="alpha2" value="${-pi/2}"/>
@@ -304,5 +304,5 @@
       <child link="link3"/>
       <origin xyz="${a4} 0 0" rpy="0 0 0"/>
-      <limit upper="2.3" lower="-2.3" effort="10000000" velocity="46"/>
+      <limit upper="2.0" lower="-2.0" effort="10000000" velocity="46"/>
       <axis xyz="0 0 1" />
     </joint>

File: aerial_manipulators_description/urdf/wp_manipulator_3R_moveit.base.urdf.xacro (robot description, xacro)
@@ -1,4 +1,4 @@
 <?xml version="1.0"?>
-<robot name="wp_manipulator" xmlns:xacro="http://ros.org/wiki/xacro">
+<robot name="wp_manipulator_3R" xmlns:xacro="http://ros.org/wiki/xacro">
   <xacro:include filename="$(find aerial_manipulators_description)/urdf/manipulator_base.urdf.xacro" />
   <link name="world"></link>
@@ -19,11 +19,3 @@
     joint_name="joint3">
   </xacro:transmisija>
-  <xacro:transmisija
-    trans_number="4"
-    joint_name="joint4">
-  </xacro:transmisija>
-  <xacro:transmisija
-    trans_number="5"
-    joint_name="joint5">
-  </xacro:transmisija>
 </robot>

Commit message: changed name to smallcase r

File: aerial_manipulators_description/urdf/manipulator_base.urdf.xacro (robot description, xacro)
@@ -181,5 +181,5 @@
     </joint>
   </xacro:macro>
-  <xacro:macro name="wp_manipulator_3R"
+  <xacro:macro name="wp_manipulator_3r"
   params="parent *origin">
     <xacro:property name="a0" value="0.04526"/>
@@ -290,5 +290,5 @@
       <!-- Adjust Gazebo coordinate system to link1 coordinate system -->
       <origin xyz="0 0 0" rpy="0 0 0"/>
-      <limit upper="1.57" lower="-1.57" effort="10000000" velocity="46"/>
+      <limit upper="1.57" lower="-0.25" effort="10000000" velocity="46"/>
       <axis xyz="0 0 1" />
     </joint>
@@ -297,5 +297,5 @@
       <child link="link2"/>
       <origin xyz="0 ${a2} 0" rpy="${-pi/2} 0 ${pi/2}"/>
-      <limit upper="2.0" lower="-2.0" effort="10000000" velocity="46"/>
+      <limit upper="1.57" lower="-1.57" effort="10000000" velocity="46"/>
       <axis xyz="0 0 1" />
     </joint>
@@ -304,5 +304,5 @@
       <child link="link3"/>
       <origin xyz="${a4} 0 0" rpy="0 0 0"/>
-      <limit upper="2.0" lower="-2.0" effort="10000000" velocity="46"/>
+      <limit upper="1.57" lower="-1.57" effort="10000000" velocity="46"/>
       <axis xyz="0 0 1" />
     </joint>

File: aerial_manipulators_description/urdf/wp_manipulator_3r.base.urdf.xacro (robot description, xacro)
@@ -1,10 +1,10 @@
 <?xml version="1.0"?>
-<robot name="wp_manipulator_3R" xmlns:xacro="http://ros.org/wiki/xacro">
+<robot name="wp_manipulator_3r" xmlns:xacro="http://ros.org/wiki/xacro">
   <xacro:include filename="$(find aerial_manipulators_description)/urdf/manipulator_base.urdf.xacro" />
   <link name="world"></link>
-  <xacro:wp_manipulator_3R
+  <xacro:wp_manipulator_3r
     parent="world">
-    <origin xyz="0 0 0" rpy="0 0 0"/>
-  </xacro:wp_manipulator_3R>
+    <origin xyz="0 0 0.035" rpy="${pi/2} 0 ${pi}"/>
+  </xacro:wp_manipulator_3r>
    <xacro:transmisija
     trans_number="1"

File: aerial_manipulators_description/urdf/wp_manipulator_3r.gazebo.xacro (robot description, xacro)
@@ -1,4 +1,4 @@
 <?xml version="1.0"?>
-<robot name="wp_manipulator_3R" xmlns:xacro="http://ros.org/wiki/xacro">
+<robot name="wp_manipulator_3r" xmlns:xacro="http://ros.org/wiki/xacro">
   <!--
   It seems that the xacro:property does not allow to use substitution args. Therefore, instead xacro parameter ${namespace}, subsitution argument is used $(arg name). This is<
@@ -6,10 +6,10 @@
   -->
   <xacro:property name="enable_bag_plugin" value="false" />
-  <xacro:property name="bag_file" value="wp_manipulator_3R.bag" />
+  <xacro:property name="bag_file" value="wp_manipulator_3r.bag" />
   <!-- Instantiate cmanip "mechanics" -->
-  <xacro:include filename="$(find aerial_manipulators_description)/urdf/wp_manipulator_3R.base.urdf.xacro" />
+  <xacro:include filename="$(find aerial_manipulators_description)/urdf/wp_manipulator_3r.base.urdf.xacro" />
   <gazebo>
     <plugin name="gazebo_ros_control" filename="libgazebo_ros_control.so">
-      <robotNamespace>/wp_manipulator_3R</robotNamespace>
+      <robotNamespace>/wp_manipulator_3r</robotNamespace>
     </plugin>
   </gazebo>

File: aerial_manipulators_description/urdf/wp_manipulator_3r_moveit.base.urdf.xacro (robot description, xacro)
@@ -1,10 +1,10 @@
 <?xml version="1.0"?>
-<robot name="wp_manipulator_3R" xmlns:xacro="http://ros.org/wiki/xacro">
+<robot name="wp_manipulator_3r" xmlns:xacro="http://ros.org/wiki/xacro">
   <xacro:include filename="$(find aerial_manipulators_description)/urdf/manipulator_base.urdf.xacro" />
   <link name="world"></link>
-  <xacro:wp_manipulator_3R
+  <xacro:wp_manipulator_3r
     parent="world">
-    <origin xyz="0 0 0.035" rpy="${pi/2} 0 ${pi}"/>
-  </xacro:wp_manipulator_3R>
+    <origin xyz="0 0 0" rpy="0 0 0"/>
+  </xacro:wp_manipulator_3r>
    <xacro:transmisija
     trans_number="1"

Commit message: added force sensor on manipulator

File: aerial_manipulators_description/urdf/manipulator_base.urdf.xacro (robot description, xacro)
@@ -175,9 +175,32 @@
       <axis xyz="0 0 1" />
     </joint>
-    <joint name="jointEndEffectorBase" type="fixed">
+    <joint name="jointEndEffectorBase" type="prismatic">
       <parent link="link5"/>
       <child link="end_effector_base"/>
       <origin xyz="${d5} 0 0" rpy="0 0 0"/>
-    </joint>
+      <axis xyz="1 0 0" />
+      <limit effort="0" velocity="0" lower="0" upper="0" />
+    </joint>
+    <!-- Enable the Joint Feedback -->
+    <gazebo reference="jointEndEffectorBase">
+      <stopCfm>0.08</stopCfm>
+      <stopErp>0.2</stopErp>
+      <implicitSpringDamper>true</implicitSpringDamper>
+      <provideFeedback>true</provideFeedback>
+    </gazebo>
+    <!-- The ft_sensor plugin  -->
+    <gazebo>
+      <plugin name="ft_sensor" filename="libgazebo_ros_ft_sensor.so">
+        <updateRate>1000.0</updateRate>
+        <robotNamespace>$(arg name)/wp_manipulator</robotNamespace>
+        <topicName>force_sensor/ft_sensor</topicName>
+        <jointName>jointEndEffectorBase</jointName>
+        <noise>
+          <type>gaussian</type>
+          <mean>0.0</mean>
+          <stddev>0.0001</stddev> <!-- change this to simulate noise -->
+        </noise>
+      </plugin>
+    </gazebo>
   </xacro:macro>
   <xacro:macro name="wp_manipulator_3r"

Commit message: changed moveit files

File: aerial_manipulators_description/urdf/manipulator_base.urdf.xacro (robot description, xacro)
@@ -1,6 +1,5 @@
 <?xml version="1.0"?>
 <robot xmlns:xacro="http://ros.org/wiki/xacro">
-  <xacro:macro name="wp_manipulator"
-  params="parent *origin">
+  <xacro:macro name="wp_manipulator" params="parent *origin">
     <xacro:property name="a0" value="0.04526"/>
     <xacro:property name="a1" value="0.122490"/>
@@ -182,25 +181,4 @@
       <limit effort="0" velocity="0" lower="0" upper="0" />
     </joint>
-    <!-- Enable the Joint Feedback -->
-    <gazebo reference="jointEndEffectorBase">
-      <stopCfm>0.08</stopCfm>
-      <stopErp>0.2</stopErp>
-      <implicitSpringDamper>true</implicitSpringDamper>
-      <provideFeedback>true</provideFeedback>
-    </gazebo>
-    <!-- The ft_sensor plugin  -->
-    <gazebo>
-      <plugin name="ft_sensor" filename="libgazebo_ros_ft_sensor.so">
-        <updateRate>1000.0</updateRate>
-        <robotNamespace>$(arg name)/wp_manipulator</robotNamespace>
-        <topicName>force_sensor/ft_sensor</topicName>
-        <jointName>jointEndEffectorBase</jointName>
-        <noise>
-          <type>gaussian</type>
-          <mean>0.0</mean>
-          <stddev>0.0001</stddev> <!-- change this to simulate noise -->
-        </noise>
-      </plugin>
-    </gazebo>
   </xacro:macro>
   <xacro:macro name="wp_manipulator_3r"

Commit message: added aerial manipulator control

File: aerial_manipulators_description/urdf/manipulator_base.urdf.xacro (robot description, xacro)
@@ -174,10 +174,10 @@
       <axis xyz="0 0 1" />
     </joint>
-    <joint name="jointEndEffectorBase" type="prismatic">
+    <joint name="jointEndEffectorBase" type="fixed">
       <parent link="link5"/>
       <child link="end_effector_base"/>
       <origin xyz="${d5} 0 0" rpy="0 0 0"/>
-      <axis xyz="1 0 0" />
-      <limit effort="0" velocity="0" lower="0" upper="0" />
+      <!--axis xyz="1 0 0" />
+      <limit effort="0" velocity="0" lower="0" upper="0" /-->
     </joint>
   </xacro:macro>
