Commit message: added new manipulator type

File: aerial_manipulators_description/urdf/manipulator_base.urdf.xacro (robot description, xacro)
@@ -181,4 +181,135 @@
     </joint>
   </xacro:macro>
+  <xacro:macro name="wp_manipulator_3rx"
+  params="parent *origin">
+    <xacro:property name="a0" value="0.04526"/>
+    <xacro:property name="a1" value="0.122490"/>
+    <xacro:property name="a2" value="0.1365"/>
+    <xacro:property name="a3" value="0.075511"/>
+    <xacro:property name="a4" value="0.072489"/>
+    <xacro:property name="d5" value="0.04526"/>
+    <xacro:property name="theta1" value="${pi/2}"/>
+    <xacro:property name="alpha2" value="${-pi/2}"/>
+    <xacro:property name="mass2" value="0.03"/>
+    <xacro:property name="mass1" value="${mass2*a1/a2}"/>
+    <xacro:property name="mass3" value="${mass2*a3/a2}"/>
+    <xacro:property name="mass4" value="${mass2*a4/a2}"/>
+    <xacro:property name="mass5" value="${mass2*d5/a2}"/>
+    <xacro:property name="rad" value="0.03"/>
+    <link name='base'>
+      <inertial>
+        <mass value="${mass5}" />
+        <origin xyz="0 -${a0/2} 0" rpy="0 0 0"/>
+        <inertia
+          ixx="${1/2 * mass5 * rad * rad}" ixy="0" ixz="0"
+          iyx="0" iyy="${1/12 * mass5 * (3*rad*rad + a0*a0)}" iyz="0"
+          izx="0" izy="0" izz="${1/12 * mass5 * (3*rad*rad + a0*a0)}"/>
+      </inertial>
+      <visual>
+        <origin xyz="0 0 0" rpy="0 0 0" />
+        <geometry>
+          <mesh filename="package://aerial_manipulators_description/meshes/wp_manipulator/base.dae"
+            scale="1 1 1" />
+        </geometry>
+      </visual>
+    </link>
+    <link name='link1'>
+      <inertial>
+        <mass value="${mass3}" />
+        <origin xyz="${a3/2} 0 0" rpy="0 0 0"/>
+        <inertia
+          ixx="${1/2 * mass3 * rad * rad}" ixy="0" ixz="0"
+          iyx="0" iyy="${1/12 * mass3 * (3*rad*rad + a3*a3)}" iyz="0"
+          izx="0" izy="0" izz="${1/12 * mass3 * (3*rad*rad + a3*a3)}"/>
+      </inertial>
+      <visual>
+        <origin xyz="0 0 0" rpy="0 ${pi / 2} ${-pi / 2}" />
+        <geometry>
+          <mesh filename="package://aerial_manipulators_description/meshes/wp_manipulator/link3.dae"
+            scale="1 1 1" />
+        </geometry>
+      </visual>
+    </link>
+    <link name='link2'>
+      <inertial>
+        <mass value="${mass4}" />
+        <origin xyz="${a4/2} 0 0" rpy="0 0 0"/>
+        <inertia
+          ixx="${1/2 * mass4 * rad * rad}" ixy="0" ixz="0"
+          iyx="0" iyy="${1/12 * mass4 * (3*rad*rad + a4*a4)}" iyz="0"
+          izx="0" izy="0" izz="${1/12 * mass4 * (3*rad*rad + a4*a4)}"/>
+      </inertial>
+      <visual>
+        <origin xyz="0 0 0" rpy="0 ${pi / 2} -${pi / 2}" />
+        <geometry>
+          <mesh filename="package://aerial_manipulators_description/meshes/wp_manipulator/link4.dae"
+            scale="1 1 1" />
+        </geometry>
+      </visual>
+    </link>
+    <link name='link3'>
+      <inertial>
+        <mass value="${mass5}" />
+        <origin xyz="${d5/2} 0 0" rpy="0 0 0"/>
+        <inertia
+          ixx="${1/2 * mass5 * rad * rad}" ixy="0" ixz="0"
+          iyx="0" iyy="${1/12 * mass5 * (3*rad*rad + d5*d5)}" iyz="0"
+          izx="0" izy="0" izz="${1/12 * mass5 * (3*rad*rad + d5*d5)}"/>
+      </inertial>
+      <visual>
+        <origin xyz="0 0 0" rpy="0 ${pi / 2} 0" />
+        <geometry>
+          <mesh filename="package://aerial_manipulators_description/meshes/wp_manipulator/link5.dae"
+            scale="1 1 1" />
+        </geometry>
+      </visual>
+    </link>
+    <link name='end_effector_base'>
+      <inertial>
+        <mass value="0.00001" />
+        <origin xyz="0 0 0" rpy="0 0 0"/>
+        <inertia
+          ixx="0.00001" ixy="0" ixz="0"
+          iyx="0" iyy="0.00001" iyz="0"
+          izx="0" izy="0" izz="0.00001"/>
+      </inertial>
+      <visual>
+        <geometry>
+          <sphere radius="0.005"/>
+        </geometry>
+      </visual>
+    </link>
+    <joint name="wp_base_joint" type="fixed">
+      <parent link="${parent}"/>
+      <child link="base"/>
+      <xacro:insert_block name="origin"/>
+    </joint>
+    <joint name="joint1" type="revolute">
+      <parent link="base"/>
+      <child link="link1"/>
+      <origin xyz="${a2} 0 0" rpy="${alpha2} 0 0"/>
+      <limit upper="1.57" lower="-1.57" effort="10000000" velocity="46"/>
+      <axis xyz="0 0 1" />
+    </joint>
+    <joint name="joint2" type="revolute">
+      <parent link="link1"/>
+      <child link="link2"/>
+      <origin xyz="${a3} 0 0" rpy="0 0 0"/>
+      <limit upper="2.0" lower="-2.0" effort="10000000" velocity="46"/>
+      <axis xyz="0 0 1" />
+    </joint>
+    <joint name="joint3" type="revolute">
+      <parent link="link2"/>
+      <child link="link3"/>
+      <origin xyz="${a4} 0 0" rpy="0 0 0"/>
+      <limit upper="2.3" lower="-2.3" effort="10000000" velocity="46"/>
+      <axis xyz="0 0 1" />
+    </joint>
+    <joint name="jointEndEffectorBase" type="fixed">
+      <parent link="link3"/>
+      <child link="end_effector_base"/>
+      <origin xyz="${d5} 0 0" rpy="0 0 0"/>
+    </joint>
+  </xacro:macro>
   <xacro:macro name="wp_manipulator_3r"
   params="parent *origin">

Commit message: added new manipulator 3rx

File: aerial_manipulators_description/urdf/manipulator_base.urdf.xacro (robot description, xacro)
@@ -200,15 +200,15 @@
     <link name='base'>
       <inertial>
-        <mass value="${mass5}" />
-        <origin xyz="0 -${a0/2} 0" rpy="0 0 0"/>
-        <inertia
-          ixx="${1/2 * mass5 * rad * rad}" ixy="0" ixz="0"
-          iyx="0" iyy="${1/12 * mass5 * (3*rad*rad + a0*a0)}" iyz="0"
-          izx="0" izy="0" izz="${1/12 * mass5 * (3*rad*rad + a0*a0)}"/>
-      </inertial>
-      <visual>
-        <origin xyz="0 0 0" rpy="0 0 0" />
-        <geometry>
-          <mesh filename="package://aerial_manipulators_description/meshes/wp_manipulator/base.dae"
+        <mass value="${mass2}" />
+        <origin xyz="${a2/2} 0 0" rpy="0 0 0"/>
+        <inertia
+          ixx="${1/2 * mass2 * rad * rad}" ixy="0" ixz="0"
+          iyx="0" iyy="${1/12 * mass2 * (3*rad*rad + a2*a2)}" iyz="0"
+          izx="0" izy="0" izz="${1/12 * mass2 * (3*rad*rad + a2*a2)}"/>
+      </inertial>
+      <visual>
+        <origin xyz="0 0 0" rpy="0 0 -${pi / 2}" />
+        <geometry>
+          <mesh filename="package://aerial_manipulators_description/meshes/wp_manipulator/link2.dae"
             scale="1 1 1" />
         </geometry>

Commit message: addded pi in xacro file

File: aerial_manipulators_description/urdf/manipulator_base.urdf.xacro (robot description, xacro)
@@ -1,4 +1,5 @@
 <?xml version="1.0"?>
 <robot xmlns:xacro="http://ros.org/wiki/xacro">
+  <xacro:property name="pi" value="3.1415926535897931" />
   <xacro:macro name="wp_manipulator" params="parent *origin">
     <xacro:property name="a0" value="0.04526"/>

Commit message: addded pi in xacro file

File: aerial_manipulators_description/urdf/manipulator_base.urdf.xacro (robot description, xacro)
@@ -2,4 +2,5 @@
 <robot xmlns:xacro="http://ros.org/wiki/xacro">
   <xacro:property name="pi" value="3.1415926535897931" />
+  <xacro:property name="mass2" value="0.03"/>
   <xacro:macro name="wp_manipulator" params="parent *origin">
     <xacro:property name="a0" value="0.04526"/>

Commit message: addded pi in xacro file

File: aerial_manipulators_description/urdf/manipulator_base.urdf.xacro (robot description, xacro)
@@ -2,5 +2,17 @@
 <robot xmlns:xacro="http://ros.org/wiki/xacro">
   <xacro:property name="pi" value="3.1415926535897931" />
+  <xacro:property name="a0" value="0.04526"/>
+  <xacro:property name="a1" value="0.122490"/>
+  <xacro:property name="a2" value="0.1365"/>
+  <xacro:property name="a3" value="0.075511"/>
+  <xacro:property name="a4" value="0.072489"/>
+  <xacro:property name="d5" value="0.04526"/>
+  <xacro:property name="theta1" value="${pi/2}"/>
+  <xacro:property name="alpha2" value="${-pi/2}"/>
   <xacro:property name="mass2" value="0.03"/>
+  <xacro:property name="mass1" value="${mass2*a1/a2}"/>
+  <xacro:property name="mass3" value="${mass2*a3/a2}"/>
+  <xacro:property name="mass4" value="${mass2*a4/a2}"/>
+  <xacro:property name="mass5" value="${mass2*d5/a2}"/>
   <xacro:macro name="wp_manipulator" params="parent *origin">
     <xacro:property name="a0" value="0.04526"/>

Commit message: addded pi in xacro file

File: aerial_manipulators_description/urdf/manipulator_base.urdf.xacro (robot description, xacro)
@@ -15,4 +15,5 @@
   <xacro:property name="mass4" value="${mass2*a4/a2}"/>
   <xacro:property name="mass5" value="${mass2*d5/a2}"/>
+  <xacro:property name="rad" value="0.03"/>
   <xacro:macro name="wp_manipulator" params="parent *origin">
     <xacro:property name="a0" value="0.04526"/>

Commit message: addded pi in xacro file

File: aerial_manipulators_description/urdf/manipulator_base.urdf.xacro (robot description, xacro)
@@ -1,19 +1,4 @@
 <?xml version="1.0"?>
 <robot xmlns:xacro="http://ros.org/wiki/xacro">
-  <xacro:property name="pi" value="3.1415926535897931" />
-  <xacro:property name="a0" value="0.04526"/>
-  <xacro:property name="a1" value="0.122490"/>
-  <xacro:property name="a2" value="0.1365"/>
-  <xacro:property name="a3" value="0.075511"/>
-  <xacro:property name="a4" value="0.072489"/>
-  <xacro:property name="d5" value="0.04526"/>
-  <xacro:property name="theta1" value="${pi/2}"/>
-  <xacro:property name="alpha2" value="${-pi/2}"/>
-  <xacro:property name="mass2" value="0.03"/>
-  <xacro:property name="mass1" value="${mass2*a1/a2}"/>
-  <xacro:property name="mass3" value="${mass2*a3/a2}"/>
-  <xacro:property name="mass4" value="${mass2*a4/a2}"/>
-  <xacro:property name="mass5" value="${mass2*d5/a2}"/>
-  <xacro:property name="rad" value="0.03"/>
   <xacro:macro name="wp_manipulator" params="parent *origin">
     <xacro:property name="a0" value="0.04526"/>

Commit message: working asap_manipulator

File: aerial_manipulators_description/urdf/manipulator_base.urdf.xacro (robot description, xacro)
@@ -514,7 +514,7 @@
     <link name="link5">
       <inertial>
-       <mass value="0.073"/>
+       <mass value="0.0073"/>
         <origin rpy="0 0 0" xyz="0.01488432 0.0 -0.00013634"/>
-        <inertia ixx="0.00001754" ixy="0.0" ixz="-0.00000035" iyx="0.0" iyy="0.00003064" iyz="0.0" izx="-0.00000035" izy="0.0" izz="0.00002513"/>
+        <inertia ixx="0.0000001754" ixy="0.0" ixz="-0.0000000035" iyx="0.0" iyy="0.0000003064" iyz="0.0" izx="-0.0000000035" izy="0.0" izz="0.0000002513"/>
       </inertial>
       <visual>

Commit message: added two versions of ASAP manipulator, 5 and 4 joints

File: aerial_manipulators_description/urdf/manipulator_base.urdf.xacro (robot description, xacro)
@@ -589,4 +589,109 @@
     </joint>
   </xacro:macro>
+  <xacro:macro name="asap_manipulator_4r"
+  params="parent *origin">
+    <link name="link1">
+      <inertial>
+        <mass value="0.124"/>
+        <origin rpy="0 0 0" xyz="0.04579089 0.00000307 -0.00007578"/>
+        <inertia ixx="0.00005883" ixy="0.0" ixz="-0.00000004" iyx="0.0" iyy="0.00032946" iyz="0.0" izx="-0.00000004" izy="0.0" izz="0.00033468"/>
+      </inertial>
+      <visual>
+        <origin rpy="0 0 0" xyz="0.0 0.0 0.0"/>
+        <geometry>
+          <mesh filename="package://aerial_manipulators_description/meshes/asap_manipulator/link2.dae" scale="1 1 1"/>
+        </geometry>
+      </visual>
+    </link>
+    <link name="link2">
+      <inertial>
+        <mass value="0.154"/>
+        <origin rpy="0 0 0" xyz="0.05074787 -0.00000371 -0.00012646"/>
+        <inertia ixx="0.00003915" ixy="0.0" ixz="0.0" iyx="0.0" iyy="0.00025748" iyz="0.0" izx="0.0" izy="0.0" izz="0.00024598"/>
+      </inertial>
+      <visual>
+       <origin rpy="0 0 0" xyz="0.0 0.0 0.0"/>
+       <geometry>
+         <mesh filename="package://aerial_manipulators_description/meshes/asap_manipulator/link3.dae" scale="1 1 1"/>
+       </geometry>
+      </visual>
+    </link>
+    <link name="link3">
+      <inertial>
+       <mass value="0.03253"/>
+        <origin rpy="0 0 0" xyz="0.07550004 0.0 0.0"/>
+        <inertia ixx="0.00002461" ixy="0.0" ixz="0.0" iyx="0.0" iyy="0.00007186" iyz="0.0" izx="0.0" izy="0.0" izz="0.00006467"/>
+      </inertial>
+      <visual>
+       <origin rpy="0 0 0" xyz="0.0 0.0 0.0"/>
+       <geometry>
+         <mesh filename="package://aerial_manipulators_description/meshes/asap_manipulator/link4.dae" scale="1 1 1"/>
+       </geometry>
+      </visual>
+    </link>
+    <link name="link4">
+      <inertial>
+       <mass value="0.0073"/>
+        <origin rpy="0 0 0" xyz="0.01488432 0.0 -0.00013634"/>
+        <inertia ixx="0.0000001754" ixy="0.0" ixz="-0.0000000035" iyx="0.0" iyy="0.0000003064" iyz="0.0" izx="-0.0000000035" izy="0.0" izz="0.0000002513"/>
+      </inertial>
+      <visual>
+       <origin rpy="0 0 0" xyz="0.0 0.0 0.0"/>
+       <geometry>
+         <mesh filename="package://aerial_manipulators_description/meshes/asap_manipulator/link5.dae" scale="1 1 1"/>
+       </geometry>
+      </visual>
+    </link>
+    <link name='end_effector_base'>
+      <inertial>
+        <mass value="0.00001" />
+        <origin xyz="0 0 0" rpy="0 0 0"/>
+        <inertia
+          ixx="0.00001" ixy="0" ixz="0"
+          iyx="0" iyy="0.00001" iyz="0"
+          izx="0" izy="0" izz="0.00001"/>
+      </inertial>
+      <visual>
+        <geometry>
+          <sphere radius="0.005"/>
+        </geometry>
+      </visual>
+    </link>
+    <joint name="joint1" type="revolute">
+      <parent link="${parent}"/>
+      <child link="link1"/>
+      <xacro:insert_block name="origin"/>
+      <limit upper="2.0" lower="-2.0" effort="10000000" velocity="46"/>
+      <axis xyz="0 0 1" />
+    </joint>
+    <joint name="joint2" type="revolute">
+      <parent link="link1"/>
+      <child link="link2"/>
+      <origin xyz="0.17955 0 0" rpy="${pi/2} 0 0"/>
+      <limit upper="1.57" lower="-1.57" effort="10000000" velocity="46"/>
+      <axis xyz="0 0 1" />
+    </joint>
+    <joint name="joint3" type="revolute">
+      <parent link="link2"/>
+      <child link="link3"/>
+      <origin xyz="0.1015 0 0" rpy="0 0 0"/>
+      <limit upper="2.0" lower="-2.0" effort="10000000" velocity="46"/>
+      <axis xyz="0 0 1" />
+    </joint>
+    <joint name="joint4" type="revolute">
+      <parent link="link3"/>
+      <child link="link4"/>
+      <origin xyz="0.151 0 0" rpy="0 0 0"/>
+      <limit upper="2.3" lower="-2.3" effort="10000000" velocity="46"/>
+      <axis xyz="0 0 1" />
+    </joint>
+    <joint name="jointEndEffectorBase" type="fixed">
+      <parent link="link4"/>
+      <child link="end_effector_base"/>
+      <origin xyz="0.048 0 0" rpy="0 0 0"/>
+      <!--axis xyz="1 0 0" />
+      <limit effort="0" velocity="0" lower="0" upper="0" /-->
+    </joint>
+  </xacro:macro>
   <!-- We add a <transmission> block for every joint that we wish to actuate. -->
   <xacro:macro name="transmisija" params="trans_number joint_name">

Commit message: new manipulator added to the package

File: aerial_manipulators_description/urdf/manipulator_base.urdf.xacro (robot description, xacro)
@@ -589,4 +589,128 @@
     </joint>
   </xacro:macro>
+  <xacro:macro name="asap_manipulator_4r_reversed" params="parent *origin">
+    <link name="link1">
+      <inertial>
+        <mass value="0.124"/>
+        <origin rpy="${pi/2} ${pi} 0" xyz="0.089775 0.00000307 -0.00007578"/>
+        <inertia ixx="0.00005883" ixy="0.0" ixz="-0.00000004" iyx="0.0" iyy="0.00032946" iyz="0.0" izx="-0.00000004" izy="0.0" izz="0.00033468"/>
+      </inertial>
+      <visual>
+        <origin rpy="${pi/2} ${pi} 0" xyz="0.17955 0.0 0.0"/>
+        <geometry>
+          <mesh filename="package://aerial_manipulators_description/meshes/asap_manipulator/link2.dae" scale="1 1 1"/>
+        </geometry>
+      </visual>
+    </link>
+    <link name="link2">
+      <inertial>
+        <mass value="0.154"/>
+        <origin rpy="0 0 0" xyz="0.05074787 -0.00000371 -0.00012646"/>
+        <inertia ixx="0.00003915" ixy="0.0" ixz="0.0" iyx="0.0" iyy="0.00025748" iyz="0.0" izx="0.0" izy="0.0" izz="0.00024598"/>
+      </inertial>
+      <visual>
+       <origin rpy="0 0 0" xyz="0.0 0.0 0.0"/>
+       <geometry>
+         <mesh filename="package://aerial_manipulators_description/meshes/asap_manipulator/link3.dae" scale="1 1 1"/>
+       </geometry>
+      </visual>
+    </link>
+    <link name="link3">
+      <inertial>
+       <mass value="0.03253"/>
+        <origin rpy="0 0 0" xyz="0.07550004 0.0 0.0"/>
+        <inertia ixx="0.00002461" ixy="0.0" ixz="0.0" iyx="0.0" iyy="0.00007186" iyz="0.0" izx="0.0" izy="0.0" izz="0.00006467"/>
+      </inertial>
+      <visual>
+       <origin rpy="0 0 0" xyz="0.0 0.0 0.0"/>
+       <geometry>
+         <mesh filename="package://aerial_manipulators_description/meshes/asap_manipulator/link4.dae" scale="1 1 1"/>
+       </geometry>
+      </visual>
+    </link>
+    <link name="link4">
+      <inertial>
+       <mass value="0.0073"/>
+        <origin rpy="${pi} ${pi} 0" xyz="0.048 0.0 -0.00013634"/>
+        <inertia ixx="0.0000001754" ixy="0.0" ixz="-0.0000000035" iyx="0.0" iyy="0.0000003064" iyz="0.0" izx="-0.0000000035" izy="0.0" izz="0.0000002513"/>
+      </inertial>
+      <visual>
+       <origin rpy="${pi} ${pi} 0" xyz="0.048 0.0 0.0"/>
+       <geometry>
+         <mesh filename="package://aerial_manipulators_description/meshes/asap_manipulator/link5.dae" scale="1 1 1"/>
+       </geometry>
+      </visual>
+    </link>
+    <link name='end_effector_base'>
+      <inertial>
+        <mass value="0.00001" />
+        <origin xyz="0 0 0" rpy="0 0 0"/>
+        <inertia
+          ixx="0.00001" ixy="0" ixz="0"
+          iyx="0" iyy="0.00001" iyz="0"
+          izx="0" izy="0" izz="0.00001"/>
+      </inertial>
+      <visual>
+        <geometry>
+          <sphere radius="0.005"/>
+        </geometry>
+      </visual>
+    </link>
+    <link name='end_effector'>
+      <inertial>
+        <mass value="0.00001" />
+        <origin xyz="0 0 0" rpy="0 0 0"/>
+        <inertia
+          ixx="0.00001" ixy="0" ixz="0"
+          iyx="0" iyy="0.00001" iyz="0"
+          izx="0" izy="0" izz="0.00001"/>
+      </inertial>
+      <visual>
+        <geometry>
+          <sphere radius="0.005"/>
+        </geometry>
+      </visual>
+    </link>
+    <joint name="jointBaseArm" type="fixed">
+      <parent link="${parent}"/>
+      <child link="link4"/>
+      <xacro:insert_block name="origin"/>
+    </joint>
+    <joint name="joint1" type="revolute">
+      <parent link="link4"/>
+      <child link="link3"/>
+      <origin xyz="0.048 0 0" rpy="0 0 0"/>
+      <limit upper="2.0" lower="-2.0" effort="10000000" velocity="46"/>
+      <axis xyz="0 0 1" />
+    </joint>
+    <joint name="joint2" type="revolute">
+      <parent link="link3"/>
+      <child link="link2"/>
+      <origin xyz="0.151 0 0" rpy="0 0 0"/>
+      <limit upper="1.57" lower="-1.57" effort="10000000" velocity="46"/>
+      <axis xyz="0 0 1" />
+    </joint>
+    <joint name="joint3" type="revolute">
+      <parent link="link2"/>
+      <child link="link1"/>
+      <origin xyz="0.1015 0 0" rpy="0 0 0"/>
+      <limit upper="2.0" lower="-2.0" effort="10000000" velocity="46"/>
+      <axis xyz="0 0 1" />
+    </joint>
+    <joint name="joint4" type="revolute">
+      <parent link="link1"/>
+      <child link="end_effector_base"/>
+      <origin xyz="0.17955 0 0" rpy="${pi/2} 0 0"/>
+      <limit upper="2.3" lower="-2.3" effort="10000000" velocity="46"/>
+      <axis xyz="0 0 1" />
+    </joint>
+    <joint name="jointEndEffectorBase" type="fixed">
+      <parent link="end_effector_base"/>
+      <child link="end_effector"/>
+      <origin xyz="0.048 0 0" rpy="0 0 0"/> /-->
+      <!--axis xyz="1 0 0" />
+      <limit effort="0" velocity="0" lower="0" upper="0" /-->
+    </joint>
+  </xacro:macro>
   <xacro:macro name="asap_manipulator_4r"
   params="parent *origin">
