Commit message: Enabled only 2 links

File: urdf/cmanip.base.urdf.xacro (robot description, xacro)
@@ -14,5 +14,5 @@
     joint_name="link1_to_link2">
   </xacro:transmisija>
-  <xacro:transmisija
+  <!-- xacro:transmisija
     trans_number="3"
     joint_name="link2_to_link3">
@@ -25,4 +25,4 @@
     trans_number="5"
     joint_name="link4_to_link5">
-  </xacro:transmisija>
+  </xacro:transmisija -->
 </robot>

File: urdf/manipulator_base.urdf.xacro (robot description, xacro)
@@ -51,5 +51,5 @@
       </visual>
     </link>
-    <link name='link3'>
+    <!-- link name='link3'>
       <inertial>
         <mass value="${mass3}" />
@@ -101,5 +101,5 @@
         </geometry>
       </visual>
-    </link>
+    </link -->
     <joint name="link0_to_link1" type="revolute">
       <parent link="world"/>
@@ -107,5 +107,5 @@
       <!-- Adjust Gazebo coordinate system to link1 coordinate system -->
       <origin xyz="0 0 0" rpy="${pi/2} 0 ${pi}"/>
-      <limit upper="0" lower="0" effort="1.62" velocity="11.9"/>
+      <limit upper="2" lower="-2" effort="1.62" velocity="11.9"/>
       <axis xyz="0 0 1" />
       <dynamics friction="0.0" damping="0.0"/>
@@ -115,9 +115,9 @@
       <child link="link2"/>
       <origin xyz="0 ${a1} 0" rpy="0 0 ${theta1}"/>
-      <limit upper="0" lower="0" effort="1.62" velocity="11.9"/>
+      <limit upper="2" lower="-2" effort="1.62" velocity="11.9"/>
       <axis xyz="0 0 1" />
       <dynamics friction="0.0" damping="0.0"/>
     </joint>
-    <joint name="link2_to_link3" type="revolute">
+    <!-- joint name="link2_to_link3" type="revolute">
       <parent link="link2"/>
       <child link="link3"/>
@@ -142,5 +142,5 @@
       <axis xyz="0 0 1" />
       <dynamics friction="0.0" damping="0.0"/>
-    </joint>
+    </joint -->
   </xacro:macro>
   <!-- We add a <transmission> block for every joint that we wish to actuate. -->

Commit message: Added link3

File: urdf/cmanip.base.urdf.xacro (robot description, xacro)
@@ -14,9 +14,9 @@
     joint_name="link1_to_link2">
   </xacro:transmisija>
-  <!-- xacro:transmisija
+  <xacro:transmisija
     trans_number="3"
     joint_name="link2_to_link3">
   </xacro:transmisija>
-  <xacro:transmisija
+  <!--xacro:transmisija
     trans_number="4"
     joint_name="link3_to_link4">

File: urdf/manipulator_base.urdf.xacro (robot description, xacro)
@@ -51,5 +51,5 @@
       </visual>
     </link>
-    <!-- link name='link3'>
+    <link name='link3'>
       <inertial>
         <mass value="${mass3}" />
@@ -68,5 +68,5 @@
       </visual>
     </link>
-    <link name='link4'>
+    <!-- link name='link4'>
       <inertial>
         <mass value="${mass4}" />
@@ -119,13 +119,13 @@
       <dynamics friction="0.0" damping="0.0"/>
     </joint>
-    <!-- joint name="link2_to_link3" type="revolute">
+    <joint name="link2_to_link3" type="revolute">
       <parent link="link2"/>
       <child link="link3"/>
       <origin xyz="${a2} 0 0" rpy="${alpha2} 0 0"/>
-      <limit upper="0.0" lower="0.0" effort="1.62" velocity="11.9"/>
+      <limit upper="2" lower="-2" effort="1.62" velocity="11.9"/>
       <axis xyz="0 0 1" />
       <dynamics friction="0.0" damping="0.0"/>
     </joint>
-    <joint name="link3_to_link4" type="revolute">
+    <!--joint name="link3_to_link4" type="revolute">
       <parent link="link3"/>
       <child link="link4"/>

Commit message: Added link4

File: urdf/cmanip.base.urdf.xacro (robot description, xacro)
@@ -18,9 +18,9 @@
     joint_name="link2_to_link3">
   </xacro:transmisija>
-  <!--xacro:transmisija
+  <xacro:transmisija
     trans_number="4"
     joint_name="link3_to_link4">
   </xacro:transmisija>
-  <xacro:transmisija
+  <!-- xacro:transmisija
     trans_number="5"
     joint_name="link4_to_link5">

File: urdf/manipulator_base.urdf.xacro (robot description, xacro)
@@ -68,5 +68,5 @@
       </visual>
     </link>
-    <!-- link name='link4'>
+    <link name='link4'>
       <inertial>
         <mass value="${mass4}" />
@@ -85,5 +85,5 @@
       </visual>
     </link>
-    <link name='link5'>
+    <!--link name='link5'>
       <inertial>
         <mass value="${mass5}" />
@@ -127,13 +127,13 @@
       <dynamics friction="0.0" damping="0.0"/>
     </joint>
-    <!--joint name="link3_to_link4" type="revolute">
+    <joint name="link3_to_link4" type="revolute">
       <parent link="link3"/>
       <child link="link4"/>
       <origin xyz="${a3} 0 0" rpy="0 0 0"/>
-      <limit upper="0.0" lower="0.0" effort="3.1" velocity="11.9"/>
+      <limit upper="2" lower="-2" effort="3.1" velocity="11.9"/>
       <axis xyz="0 0 1" />
       <dynamics friction="0.0" damping="0.0"/>
     </joint>
-    <joint name="link4_to_link5" type="revolute">
+    <!--joint name="link4_to_link5" type="revolute">
       <parent link="link4"/>
       <child link="link5"/>

Commit message: Added link5

File: urdf/cmanip.base.urdf.xacro (robot description, xacro)
@@ -22,7 +22,7 @@
     joint_name="link3_to_link4">
   </xacro:transmisija>
-  <!-- xacro:transmisija
+  <xacro:transmisija
     trans_number="5"
     joint_name="link4_to_link5">
-  </xacro:transmisija -->
+  </xacro:transmisija>
 </robot>

File: urdf/manipulator_base.urdf.xacro (robot description, xacro)
@@ -7,5 +7,5 @@
     <xacro:property name="a3" value="0.075511"/>
     <xacro:property name="a4" value="0.072489"/>
-    <xacro:property name="d5" value="0.04526"/>
+    <xacro:property name="a5" value="0.04526"/>
     <xacro:property name="theta1" value="${pi/2}"/>
     <xacro:property name="alpha2" value="${-pi/2}"/>
@@ -14,5 +14,5 @@
     <xacro:property name="mass3" value="${mass2*a3/a2}"/>
     <xacro:property name="mass4" value="${mass2*a4/a2}"/>
-    <xacro:property name="mass5" value="${mass2*d5/a2}"/>
+    <xacro:property name="mass5" value="${mass2*a5/a2}"/>
     <xacro:property name="rad" value="0.03"/>
     <link name="world"></link>
@@ -85,12 +85,12 @@
       </visual>
     </link>
-    <!--link name='link5'>
+    <link name='link5'>
       <inertial>
         <mass value="${mass5}" />
-        <origin xyz="${d5/2} 0 0" rpy="0 0 0"/>
+        <origin xyz="${a5/2} 0 0" rpy="0 0 0"/>
         <inertia
           ixx="${1/2 * mass5 * rad * rad}" ixy="0" ixz="0"
-          iyx="0" iyy="${1/12 * mass5 * (3*rad*rad + d5*d5)}" iyz="0"
-          izx="0" izy="0" izz="${1/12 * mass5 * (3*rad*rad + d5*d5)}"/>
+          iyx="0" iyy="${1/12 * mass5 * (3*rad*rad + a5*a5)}" iyz="0"
+          izx="0" izy="0" izz="${1/12 * mass5 * (3*rad*rad + a5*a5)}"/>
       </inertial>
       <visual>
@@ -101,5 +101,5 @@
         </geometry>
       </visual>
-    </link -->
+    </link>
     <joint name="link0_to_link1" type="revolute">
       <parent link="world"/>
@@ -133,14 +133,14 @@
       <limit upper="2" lower="-2" effort="1.62" velocity="11.9"/>
       <axis xyz="0 0 1" />
-      <dynamics friction="0.0" damping="0.0"/>
+      <dynamics friction="0.005" damping="0.0"/>
     </joint>
-    <!--joint name="link4_to_link5" type="revolute">
+    <joint name="link4_to_link5" type="revolute">
       <parent link="link4"/>
       <child link="link5"/>
       <origin xyz="${a4} 0 0" rpy="0 0 0"/>
-      <limit upper="2.355" lower="-2.355" effort="3.1" velocity="11.9"/>
+      <limit upper="1.5" lower="-1.5" effort="1.62" velocity="11.9"/>
       <axis xyz="0 0 1" />
-      <dynamics friction="0.0" damping="0.0"/>
-    </joint -->
+      <dynamics friction="0.005" damping="0.0"/>
+    </joint>
   </xacro:macro>
   <!-- We add a <transmission> block for every joint that we wish to actuate. -->

Commit message: Use origin and parent arguments properly, reorganize launch.

File: urdf/cmanip.base.urdf.xacro (robot description, xacro)
@@ -2,7 +2,8 @@
 <robot name="cmanip" xmlns:xacro="http://ros.org/wiki/xacro">
   <xacro:include filename="$(find aerial_manipulators)/urdf/manipulator_base.urdf.xacro" />
+  <link name="world"></link>
   <xacro:cmanip
     parent="world">
-    <origin xyz="0 0 0" rpy="0 0 0"/>
+    <origin xyz="0 0 0" rpy="${pi/2} 0 ${pi}"/>
   </xacro:cmanip>
   <xacro:transmisija

File: urdf/manipulator_base.urdf.xacro (robot description, xacro)
@@ -16,5 +16,5 @@
     <xacro:property name="mass5" value="${mass2*d5/a2}"/>
     <xacro:property name="rad" value="0.03"/>
-    <link name="world"></link>
+    <!--link name="world"></link-->
     <link name='link1'>
       <inertial>
@@ -118,8 +118,9 @@
     </link>
     <joint name="link0_to_link1" type="revolute">
-      <parent link="world"/>
+      <parent link="${parent}"/>
       <child link="link1"/>
       <!-- Adjust Gazebo coordinate system to link1 coordinate system -->
-      <origin xyz="0 0 0" rpy="${pi/2} 0 ${pi}"/>
+      <!--origin xyz="0 0 0.075" rpy="${pi/2} 0 ${pi}"/-->
+      <xacro:insert_block name="origin"/>
       <limit upper="1.57" lower="-1.57" effort="10000000" velocity="20"/>
       <axis xyz="0 0 1" />

Commit message: PID adjustments

File: urdf/cmanip.base.urdf.xacro (robot description, xacro)
@@ -26,3 +26,10 @@
     joint_name="link4_to_link5">
   </xacro:transmisija>
+<!--
+  <xacro:ft_sensor_gazebo
+    name="ftSensor"
+    type="force"
+    parent="link5">
+  </xacro:ft_sensor_gazebo>
+-->
 </robot>

File: urdf/manipulator_base.urdf.xacro (robot description, xacro)
@@ -10,9 +10,9 @@
     <xacro:property name="theta1" value="${pi/2}"/>
     <xacro:property name="alpha2" value="${-pi/2}"/>
-    <xacro:property name="mass2" value="0.03"/>
-    <xacro:property name="mass1" value="${mass2*a1/a2}"/>
-    <xacro:property name="mass3" value="${mass2*a3/a2}"/>
-    <xacro:property name="mass4" value="${mass2*a4/a2}"/>
-    <xacro:property name="mass5" value="${mass2*d5/a2}"/>
+    <xacro:property name="mass1" value="0.01715"/>
+    <xacro:property name="mass2" value="0.10663"/>
+    <xacro:property name="mass3" value="0.17449"/>
+    <xacro:property name="mass4" value="0.01133"/>
+    <xacro:property name="mass5" value="0.08200"/>
     <xacro:property name="rad" value="0.03"/>
     <link name="world"></link>
@@ -20,9 +20,6 @@
       <inertial>
         <mass value="${mass1}" />
-        <origin xyz="0 ${a1/2} 0" rpy="0 0 0"/>
-        <inertia
-          ixx="${1/12 * mass1 * (3*rad*rad + a1*a1)}" ixy="0" ixz="0"
-          iyx="0" iyy="${1/2 * mass1 * rad * rad}" iyz="0"
-          izx="0" izy="0" izz="${1/12 * mass1 * (3*rad*rad + a1*a1)}"/>
+        <origin xyz="0.00073 0.06124 -0.00009" rpy="0 0 0"/>
+        <inertia ixx = "0.00003618101"	ixy = "-0.00000032742"	ixz = "0.00" iyy = "0.00000866025"	iyz = "0.00"	izz = "0.00003041429"/>
       </inertial>
       <visual>
@@ -37,9 +34,6 @@
       <inertial>
         <mass value="${mass2}" />
-        <origin xyz="${a2/2} 0 0" rpy="0 0 0"/>
-        <inertia
-          ixx="${1/2 * mass2 * rad * rad}" ixy="0" ixz="0"
-          iyx="0" iyy="${1/12 * mass2 * (3*rad*rad + a2*a2)}" iyz="0"
-          izx="0" izy="0" izz="${1/12 * mass2 * (3*rad*rad + a2*a2)}"/>
+        <origin xyz="0.0257 0.00004 0" rpy="0 0 0"/>
+        <inertia ixx="0.000025414" ixy="0.00000000062" ixz="-0.00000114006" iyy="0.00013446945" iyz="0.00000000001" izz="0.00013233260"/>
       </inertial>
       <visual>
@@ -54,9 +48,6 @@
       <inertial>
         <mass value="${mass3}" />
-        <origin xyz="${a3/2} 0 0" rpy="0 0 0"/>
-        <inertia
-          ixx="${1/2 * mass3 * rad * rad}" ixy="0" ixz="0"
-          iyx="0" iyy="${1/12 * mass3 * (3*rad*rad + a3*a3)}" iyz="0"
-          izx="0" izy="0" izz="${1/12 * mass3 * (3*rad*rad + a3*a3)}"/>
+        <origin xyz="0.03443 0 0.00018" rpy="0 0 0"/>
+        <inertia ixx="0.00003095696" ixy="0.00000000169" ixz="0" iyy="0.00016728462" iyz="0" izz="0.00015971261"/>
       </inertial>
       <visual>
@@ -71,9 +62,6 @@
       <inertial>
         <mass value="${mass4}" />
-        <origin xyz="${a4/2} 0 0" rpy="0 0 0"/>
-        <inertia
-          ixx="${1/2 * mass4 * rad * rad}" ixy="0" ixz="0"
-          iyx="0" iyy="${1/12 * mass4 * (3*rad*rad + a4*a4)}" iyz="0"
-          izx="0" izy="0" izz="${1/12 * mass4 * (3*rad*rad + a4*a4)}"/>
+        <origin xyz="0.03624 0 -0.00059" rpy="0 0 0"/>
+        <inertia ixx="0.00000540203" ixy="0" ixz="0" iyy="0.00001225566" iyz="0" izz="0.00000858285"/>
       </inertial>
       <visual>
@@ -88,9 +76,6 @@
       <inertial>
         <mass value="${mass5}" />
-        <origin xyz="${d5/2} 0 0" rpy="0 0 0"/>
-        <inertia
-          ixx="${1/2 * mass5 * rad * rad}" ixy="0" ixz="0"
-          iyx="0" iyy="${1/12 * mass5 * (3*rad*rad + d5*d5)}" iyz="0"
-          izx="0" izy="0" izz="${1/12 * mass5 * (3*rad*rad + d5*d5)}"/>
+        <origin xyz="0.01179 0 0.00023" rpy="0 0 0"/>
+        <inertia ixx="0.00001323215" ixy="0.00000000037" ixz="-0.0000019846" iyy="0.00002293047" iyz="0.0000000002" izz="0.00002030725"/>
       </inertial>
       <visual>
@@ -101,5 +86,13 @@
         </geometry>
       </visual>
+      <collision>
+        <origin xyz="0 0 0" rpy="0 ${pi / 2} 0" />
+        <geometry>
+          <mesh filename="package://aerial_manipulators/meshes/wp_manipulator/link5.dae"
+            scale="1 1 1" />
+        </geometry>
+      </collision>
     </link>
+<!--
     <link name="endEffector">
       <inertial>
@@ -117,4 +110,5 @@
       </visual>
     </link>
+-->
     <joint name="link0_to_link1" type="revolute">
       <parent link="world"/>
@@ -153,6 +147,10 @@
       <limit upper="2.3" lower="-2.3" effort="10000000" velocity="20"/>
       <axis xyz="0 0 1" />
+      <sensor name="force_torque" type="force_torque">
+        <update_rate>30</update_rate>
+      </sensor>
     </joint>
 <!--       <limit upper="2.3" lower="-2.3" effort="10000000" velocity="20"/> -->
+<!--
     <joint name="link5_to_ef" type="revolute">
       <parent link="link5"/>
@@ -162,4 +160,5 @@
       <axis xyz="0 0 1" />
     </joint>
+-->
   </xacro:macro>
   <!-- We add a <transmission> block for every joint that we wish to actuate. -->
@@ -176,3 +175,23 @@
     </transmission>
   </xacro:macro>
+<!--
+  <xacro:macro name="ft_sensor_gazebo" params="parent name type">
+    <gazebo reference="${name}_${type}_base">
+      <gravity>true</gravity>
+    </gazebo>
+    <gazebo reference="${name}_${type}_measure">
+      <gravity>true</gravity>
+    </gazebo>
+    <gazebo reference="${parent}_${name}_measure_joint">
+      <provideFeedback>true</provideFeedback>
+    </gazebo>
+    <gazebo>
+        <plugin name="${name}_ft_sensor" filename="libgazebo_ros_ft_sensor.so">
+        <updateRate>1000.0</updateRate>
+        <topicName>${parent}_${name}/ft_sensor_topic</topicName>
+        <jointName>${parent}_${name}_measure_joint</jointName>
+        </plugin>
+    </gazebo>
+  </xacro:macro>
+-->
 </robot>

Commit message: Adding Force Sensor

File: urdf/cmanip.base.urdf.xacro (robot description, xacro)
@@ -28,9 +28,7 @@
   </xacro:transmisija>
 <!--
-  <xacro:ft_sensor_gazebo
-    name="ftSensor"
-    type="force"
-    parent="link5">
-  </xacro:ft_sensor_gazebo>
+  <xacro:force_sensor>
+    <origin xyz="0 0 0" rpy="0 0 0"/>
+  </xacro:force_sensor>
 -->
 </robot>

File: urdf/cmanip.gazebo.xacro (robot description, xacro)
@@ -14,3 +14,24 @@
     </plugin>
   </gazebo>
+<gazebo reference="joint_force_sensor_mount_top">
+  <stopCfm>0.08</stopCfm>
+  <stopErp>0.2</stopErp>
+  <implicitSpringDamper>true</implicitSpringDamper>
+  <provideFeedback>true</provideFeedback>
+</gazebo>
+<!--
+<gazebo>
+  <plugin name="ft_sensor" filename="libgazebo_ros_ft_sensor.so">
+    <updateRate>1000.0</updateRate>
+    <robotNamespace>$(arg name)</robotNamespace>
+    <topicName>ft_sensor</topicName>
+    <jointName>joint_force_sensor_mount_top</jointName>
+    <noise>
+      <type>gaussian</type>
+      <mean>0.0</mean>
+      <stddev>0.0001</stddev>
+    </noise>
+  </plugin>
+</gazebo>
+-->
 </robot>

File: urdf/manipulator_base.urdf.xacro (robot description, xacro)
@@ -148,7 +148,4 @@
       <limit upper="2.3" lower="-2.3" effort="10000000" velocity="20"/>
       <axis xyz="0 0 1" />
-      <sensor name="force_torque" type="force_torque">
-        <update_rate>30</update_rate>
-      </sensor>
     </joint>
 <!--       <limit upper="2.3" lower="-2.3" effort="10000000" velocity="20"/> -->
@@ -176,23 +173,114 @@
     </transmission>
   </xacro:macro>
-<!--
-  <xacro:macro name="ft_sensor_gazebo" params="parent name type">
-    <gazebo reference="${name}_${type}_base">
-      <gravity>true</gravity>
-    </gazebo>
-    <gazebo reference="${name}_${type}_measure">
-      <gravity>true</gravity>
-    </gazebo>
-    <gazebo reference="${parent}_${name}_measure_joint">
-      <provideFeedback>true</provideFeedback>
-    </gazebo>
-    <gazebo>
-        <plugin name="${name}_ft_sensor" filename="libgazebo_ros_ft_sensor.so">
-        <updateRate>1000.0</updateRate>
-        <topicName>${parent}_${name}/ft_sensor_topic</topicName>
-        <jointName>${parent}_${name}_measure_joint</jointName>
-        </plugin>
-    </gazebo>
+  <xacro:macro name="force_sensor"
+    params="*origin">
+    <!--_____________________________________________________________-->
+    <!--LINK1 force sensor stand-->
+    <!--_____________________________________________________________-->
+    <link name='link_force_sensor_stand'>
+      <inertial>
+        <mass value="0.2" />
+        <origin rpy="0 0 0" xyz="0 0.046818651 0"/>
+        <inertia
+          ixx="0.023434322" ixy="0" ixz="0.0"
+          iyx="0" iyy="0.001547123" iyz="0"
+          izx="0.0" izy="0" izz="0.023434322"/>
+      </inertial>
+      <visual>
+        <origin xyz="0 0 0" rpy="0 0 0" />
+        <geometry>
+          <mesh filename="package://aerial_manipulators/meshes/wp_manipulator/forcesensor_stand.dae"
+            scale="0.1 0.1 0.1" />
+        </geometry>
+      </visual>
+      <!--collision name='collision'>
+        <origin xyz="0 0 0" rpy="0 0 0"/>
+        <geometry>
+          <mesh filename="package://mmuav_description/meshes/forcesensor_stand.dae"
+            scale="1 1 1" />
+        </geometry>
+      </collision-->
+    </link>
+    <!--_____________________________________________________________-->
+    <!--LINK2 force sensor mount bottom-->
+    <!--_____________________________________________________________-->
+    <link name='link_force_sensor_bottom_mount'>
+      <inertial>
+        <mass value="0.005" />
+        <origin rpy="0 0 0" xyz="0.0 0.000206111 0.0"/>
+        <inertia
+          ixx="0.000002139" ixy="0" ixz="0.0"
+          iyx="0" iyy="0.000004241" iyz="0"
+          izx="0.0" izy="0" izz="0.000002139"/>
+      </inertial>
+      <visual>
+        <origin xyz="0 0 0" rpy="0 0 0" />
+        <geometry>
+          <mesh filename="package://aerial_manipulators/meshes/wp_manipulator/forcesensor_mount_bottom.dae"
+            scale="0.1 0.1 0.1" />
+        </geometry>
+      </visual>
+      <!--collision name='collision'>
+        <origin xyz="0 0 0" rpy="0 0 0"/>
+        <geometry>
+          <mesh filename="package://mmuav_description/meshes/forcesensor_mount_bottom.dae"
+            scale="1 1 1" />
+        </geometry>
+      </collision-->
+    </link>
+    <!--_____________________________________________________________-->
+    <!--LINK2 force sensor mount top-->
+    <!--_____________________________________________________________-->
+    <link name='link_force_sensor_top_mount'>
+      <inertial>
+        <mass value="0.0080" />
+        <origin rpy="0 0 0" xyz="0 0 -0.002998408"/>
+        <inertia
+          ixx="0.000059994" ixy="0" ixz="0.0"
+          iyx="0" iyy="0.000059994" iyz="0"
+          izx="0.0" izy="0" izz="0.000119615"/>
+      </inertial>
+      <!--0.01903151 0.01661061 0.02154592-->
+      <visual>
+        <origin xyz="-0.0001903 -0.0001661 -0.0005153" rpy="0 0 0" />
+        <geometry>
+          <mesh filename="package://aerial_manipulators/meshes/wp_manipulator/forcesensor_mount_top.dae"
+            scale="0.1 0.1 0.1" />
+        </geometry>
+      </visual>
+      <collision name='collision'>
+        <origin xyz="-0.001903 -0.001661 -0.005153" rpy="0 0 0"/>
+        <geometry>
+          <mesh filename="package://aerial_manipulators/meshes/wp_manipulator/forcesensor_mount_top.dae"
+            scale="0.1 0.1 0.1" />
+        </geometry>
+      </collision>
+    </link>
+    <!--_____________________________________________________________-->
+    <!--JOINT1 FIXED force_sensor_stand-->
+    <!--_____________________________________________________________-->
+    <joint name="joint_force_sensor_stand" type="fixed">
+        <xacro:insert_block name="origin"/>
+        <parent link="link5"/>
+        <child link="link_force_sensor_stand"/>
+    </joint>
+    <!--_____________________________________________________________-->
+    <!--JOINT2 FIXED joint_force_sensor_mount_bottom-->
+    <!--_____________________________________________________________-->
+    <joint name="joint_force_sensor_mount_bottom" type="fixed">
+        <origin xyz="0 1.003 0" rpy="${pi} 0 0" />
+        <parent link="link_force_sensor_stand"/>
+        <child link="link_force_sensor_bottom_mount"/>
+    </joint>
+    <!--_____________________________________________________________-->
+    <!--JOINT2 FIXED force_sensor_mount_top-->
+    <!--_____________________________________________________________-->
+    <joint name="joint_force_sensor_mount_top" type="prismatic">
+        <origin xyz="0 0 0" rpy="${-pi/2} 0 0" />
+        <parent link="link_force_sensor_bottom_mount"/>
+        <child link="link_force_sensor_top_mount"/>
+        <axis xyz="0 0 1" />
+        <limit effort="0" velocity="0" lower="0" upper="0" />
+    </joint>
   </xacro:macro>
--->
 </robot>
