Commit message: Adding Force Sensor (WIP)

File: urdf/cmanip.base.urdf.xacro (robot description, xacro)
@@ -27,8 +27,6 @@
     joint_name="link4_to_link5">
   </xacro:transmisija>
-<!--
   <xacro:force_sensor>
-    <origin xyz="0 0 0" rpy="0 0 0"/>
+    <origin xyz="0.04526 0 0" rpy="0 0 -1.57"/>
   </xacro:force_sensor>
--->
 </robot>

File: urdf/cmanip.gazebo.xacro (robot description, xacro)
@@ -20,8 +20,7 @@
   <provideFeedback>true</provideFeedback>
 </gazebo>
-<!--
 <gazebo>
   <plugin name="ft_sensor" filename="libgazebo_ros_ft_sensor.so">
-    <updateRate>1000.0</updateRate>
+    <updateRate>10.0</updateRate>
     <robotNamespace>$(arg name)</robotNamespace>
     <topicName>ft_sensor</topicName>
@@ -34,4 +33,3 @@
   </plugin>
 </gazebo>
--->
 </robot>

File: urdf/manipulator_base.urdf.xacro (robot description, xacro)
@@ -174,113 +174,113 @@
   </xacro:macro>
   <xacro:macro name="force_sensor"
-    params="*origin">
-    <!--_____________________________________________________________-->
-    <!--LINK1 force sensor stand-->
-    <!--_____________________________________________________________-->
-    <link name='link_force_sensor_stand'>
-      <inertial>
-        <mass value="0.2" />
-        <origin rpy="0 0 0" xyz="0 0.046818651 0"/>
-        <inertia
-          ixx="0.023434322" ixy="0" ixz="0.0"
-          iyx="0" iyy="0.001547123" iyz="0"
-          izx="0.0" izy="0" izz="0.023434322"/>
-      </inertial>
-      <visual>
-        <origin xyz="0 0 0" rpy="0 0 0" />
-        <geometry>
-          <mesh filename="package://aerial_manipulators/meshes/wp_manipulator/forcesensor_stand.dae"
-            scale="0.1 0.1 0.1" />
-        </geometry>
-      </visual>
-      <!--collision name='collision'>
-        <origin xyz="0 0 0" rpy="0 0 0"/>
-        <geometry>
-          <mesh filename="package://mmuav_description/meshes/forcesensor_stand.dae"
-            scale="1 1 1" />
-        </geometry>
-      </collision-->
-    </link>
-    <!--_____________________________________________________________-->
-    <!--LINK2 force sensor mount bottom-->
-    <!--_____________________________________________________________-->
-    <link name='link_force_sensor_bottom_mount'>
-      <inertial>
-        <mass value="0.005" />
-        <origin rpy="0 0 0" xyz="0.0 0.000206111 0.0"/>
-        <inertia
-          ixx="0.000002139" ixy="0" ixz="0.0"
-          iyx="0" iyy="0.000004241" iyz="0"
-          izx="0.0" izy="0" izz="0.000002139"/>
-      </inertial>
-      <visual>
-        <origin xyz="0 0 0" rpy="0 0 0" />
-        <geometry>
-          <mesh filename="package://aerial_manipulators/meshes/wp_manipulator/forcesensor_mount_bottom.dae"
-            scale="0.1 0.1 0.1" />
-        </geometry>
-      </visual>
-      <!--collision name='collision'>
-        <origin xyz="0 0 0" rpy="0 0 0"/>
-        <geometry>
-          <mesh filename="package://mmuav_description/meshes/forcesensor_mount_bottom.dae"
-            scale="1 1 1" />
-        </geometry>
-      </collision-->
-    </link>
-    <!--_____________________________________________________________-->
-    <!--LINK2 force sensor mount top-->
-    <!--_____________________________________________________________-->
-    <link name='link_force_sensor_top_mount'>
-      <inertial>
-        <mass value="0.0080" />
-        <origin rpy="0 0 0" xyz="0 0 -0.002998408"/>
-        <inertia
-          ixx="0.000059994" ixy="0" ixz="0.0"
-          iyx="0" iyy="0.000059994" iyz="0"
-          izx="0.0" izy="0" izz="0.000119615"/>
-      </inertial>
-      <!--0.01903151 0.01661061 0.02154592-->
-      <visual>
-        <origin xyz="-0.0001903 -0.0001661 -0.0005153" rpy="0 0 0" />
-        <geometry>
-          <mesh filename="package://aerial_manipulators/meshes/wp_manipulator/forcesensor_mount_top.dae"
-            scale="0.1 0.1 0.1" />
-        </geometry>
-      </visual>
-      <collision name='collision'>
-        <origin xyz="-0.001903 -0.001661 -0.005153" rpy="0 0 0"/>
-        <geometry>
-          <mesh filename="package://aerial_manipulators/meshes/wp_manipulator/forcesensor_mount_top.dae"
-            scale="0.1 0.1 0.1" />
-        </geometry>
-      </collision>
-    </link>
-    <!--_____________________________________________________________-->
-    <!--JOINT1 FIXED force_sensor_stand-->
-    <!--_____________________________________________________________-->
-    <joint name="joint_force_sensor_stand" type="fixed">
-        <xacro:insert_block name="origin"/>
-        <parent link="link5"/>
-        <child link="link_force_sensor_stand"/>
-    </joint>
-    <!--_____________________________________________________________-->
-    <!--JOINT2 FIXED joint_force_sensor_mount_bottom-->
-    <!--_____________________________________________________________-->
-    <joint name="joint_force_sensor_mount_bottom" type="fixed">
-        <origin xyz="0 1.003 0" rpy="${pi} 0 0" />
-        <parent link="link_force_sensor_stand"/>
-        <child link="link_force_sensor_bottom_mount"/>
-    </joint>
-    <!--_____________________________________________________________-->
-    <!--JOINT2 FIXED force_sensor_mount_top-->
-    <!--_____________________________________________________________-->
-    <joint name="joint_force_sensor_mount_top" type="prismatic">
-        <origin xyz="0 0 0" rpy="${-pi/2} 0 0" />
-        <parent link="link_force_sensor_bottom_mount"/>
-        <child link="link_force_sensor_top_mount"/>
-        <axis xyz="0 0 1" />
-        <limit effort="0" velocity="0" lower="0" upper="0" />
-    </joint>
-  </xacro:macro>
+      params="*origin">
+__________________________-->
+      <!--LINK1 force sensor stand-->
+      <!--_____________________________________________________________-->
+      <link name='link_force_sensor_stand'>
+        <inertial>
+          <mass value="0.002" />
+          <origin rpy="0 0 0" xyz="0 0.46818651 0"/>
+          <inertia
+            ixx="0.00023434322" ixy="0" ixz="0.0"
+            iyx="0" iyy="0.00001547123" iyz="0"
+            izx="0.0" izy="0" izz="0.00023434322"/>
+        </inertial>
+        <visual>
+          <origin xyz="0 0 0" rpy="0 0 0" />
+          <geometry>
+            <mesh filename="package://aerial_manipulators/meshes/wp_manipulator/forcesensor_stand.dae"
+              scale="0.1 0.1 0.1" />
+          </geometry>
+        </visual>
+        <!--collision name='collision'>
+          <origin xyz="0 0 0" rpy="0 0 0"/>
+          <geometry>
+            <mesh filename="package://mmuav_description/meshes/forcesensor_stand.dae"
+              scale="1 1 1" />
+          </geometry>
+        </collision-->
+      </link>
+      <!--_____________________________________________________________-->
+      <!--LINK2 force sensor mount bottom-->
+      <!--_____________________________________________________________-->
+      <link name='link_force_sensor_bottom_mount'>
+        <inertial>
+          <mass value="0.0005" />
+          <origin rpy="0 0 0" xyz="0.0 0.000206111 0.0"/>
+          <inertia
+            ixx="0.0000002139" ixy="0" ixz="0.0"
+            iyx="0" iyy="0.0000004241" iyz="0"
+            izx="0.0" izy="0" izz="0.0000002139"/>
+        </inertial>
+        <visual>
+          <origin xyz="0 0 0" rpy="0 0 0" />
+          <geometry>
+            <mesh filename="package://aerial_manipulators/meshes/wp_manipulator/forcesensor_mount_bottom.dae"
+              scale="0.1 0.1 0.1" />
+          </geometry>
+        </visual>
+        <!--collision name='collision'>
+          <origin xyz="0 0 0" rpy="0 0 0"/>
+          <geometry>
+            <mesh filename="package://mmuav_description/meshes/forcesensor_mount_bottom.dae"
+              scale="1 1 1" />
+          </geometry>
+        </collision-->
+      </link>
+      <!--_____________________________________________________________-->
+      <!--LINK2 force sensor mount top-->
+      <!--_____________________________________________________________-->
+      <link name='link_force_sensor_top_mount'>
+        <inertial>
+          <mass value="0.00080" />
+          <origin rpy="0 0 0" xyz="0 0 -0.02998408"/>
+          <inertia
+            ixx="0.0000059994" ixy="0" ixz="0.0"
+            iyx="0" iyy="0.0000059994" iyz="0"
+            izx="0.0" izy="0" izz="0.0000119615"/>
+        </inertial>
+        <!--0.01903151 0.01661061 0.02154592-->
+        <visual>
+          <origin xyz="-0.001903 -0.001661 -0.005153" rpy="0 0 0" />
+          <geometry>
+            <mesh filename="package://aerial_manipulators/meshes/wp_manipulator/forcesensor_mount_top.dae"
+              scale="0.1 0.1 0.1" />
+          </geometry>
+        </visual>
+        <collision name='collision'>
+          <origin xyz="-0.001903 -0.001661 -0.005153" rpy="0 0 0"/>
+          <geometry>
+            <mesh filename="package://aerial_manipulators/meshes/wp_manipulator/forcesensor_mount_top.dae"
+              scale="0.1 0.1 0.1" />
+          </geometry>
+        </collision>
+      </link>
+      <!--_____________________________________________________________-->
+      <!--JOINT1 FIXED force_sensor_stand-->
+      <!--_____________________________________________________________-->
+      <joint name="joint_force_sensor_stand" type="fixed">
+          <xacro:insert_block name="origin"/>
+          <parent link="link5"/>
+          <child link="link_force_sensor_stand"/>
+      </joint>
+      <!--_____________________________________________________________-->
+      <!--JOINT2 FIXED joint_force_sensor_mount_bottom-->
+      <!--_____________________________________________________________-->
+      <joint name="joint_force_sensor_mount_bottom" type="fixed">
+          <origin xyz="0 0.1003 0" rpy="${pi} 0 0" />
+          <parent link="link_force_sensor_stand"/>
+          <child link="link_force_sensor_bottom_mount"/>
+      </joint>
+      <!--_____________________________________________________________-->
+      <!--JOINT2 FIXED force_sensor_mount_top-->
+      <!--_____________________________________________________________-->
+      <joint name="joint_force_sensor_mount_top" type="prismatic">
+          <origin xyz="0 0 0" rpy="${-pi/2} 0 0" />
+          <parent link="link_force_sensor_bottom_mount"/>
+          <child link="link_force_sensor_top_mount"/>
+          <axis xyz="0 0 1" />
+          <limit effort="0" velocity="0" lower="0" upper="0" />
+      </joint>
+    </xacro:macro>
 </robot>
