Commit message: Corrected mistakes and added inertia

File: urdf/manipulator_base.urdf.xacro (robot description, xacro)
@@ -3,16 +3,29 @@
   <xacro:macro name="cmanip"
   params="parent *origin">
+    <xacro:property name="a1" value="0.122490"/>
+    <xacro:property name="a2" value="0.136500"/>
+    <xacro:property name="a3" value="0.075511"/>
+    <xacro:property name="a4" value="0.072489"/>
+    <xacro:property name="d5" value="0.04526"/>
+    <xacro:property name="theta1" value="${pi/2}"/>
+    <xacro:property name="alpha2" value="-${pi/2}"/>
+    <xacro:property name="mass2" value="0.003"/>
+    <xacro:property name="mass1" value="${mass2*a1/a2}"/>
+    <xacro:property name="mass3" value="${mass2*a3/a2}"/>
+    <xacro:property name="mass4" value="${mass2*a4/a2}"/>
+    <xacro:property name="mass5" value="${mass2*d5/a2}"/>
+    <xacro:property name="rad" value="0.03"/>
     <link name="world"></link>
     <link name='link1'>
       <inertial>
-        <mass value="0.1" />
-        <origin xyz="0 0 0" rpy="0 0 0"/>
+        <mass value="${mass1}" />
+        <origin xyz="0 ${a1/2} 0" rpy="0 0 0"/>
         <inertia
-          ixx="0.01176" ixy="0" ixz="0"
-          iyx="0" iyy="0.01176" iyz="0"
-          izx="0" izy="0" izz="0.0252"/>
+          ixx="${1/12 * mass1 * (3*rad*rad + a1*a1)}" ixy="0" ixz="0"
+          iyx="0" iyy="${1/2 * mass1 * rad * rad}" iyz="0"
+          izx="0" izy="0" izz="${1/12 * mass1 * (3*rad*rad + a1*a1)}"/>
       </inertial>
       <visual>
-        <origin xyz="0 0 0" rpy="${- pi / 2} 0 0" />
+        <origin xyz="0 0 0" rpy="0 0 0" />
         <geometry>
           <mesh filename="package://aerial_manipulators/meshes/wp_manipulator/link1.dae"
@@ -23,13 +36,13 @@
     <link name='link2'>
       <inertial>
-        <mass value="0.1" />
-        <origin xyz="0 0 0" rpy="0 0 0"/>
+        <mass value="0.03" />
+        <origin xyz="${a2/2} 0 0" rpy="0 0 0"/>
         <inertia
-          ixx="0.01176" ixy="0" ixz="0"
-          iyx="0" iyy="0.01176" iyz="0"
-          izx="0" izy="0" izz="0.0252"/>
+          ixx="${1/2 * mass2 * rad * rad}" ixy="0" ixz="0"
+          iyx="0" iyy="${1/12 * mass2 * (3*rad*rad + a2*a2)}" iyz="0"
+          izx="0" izy="0" izz="${1/12 * mass2 * (3*rad*rad + a2*a2)}"/>
       </inertial>
       <visual>
-        <origin xyz="0 0 0" rpy="${- pi / 2} ${pi} 0" />
+        <origin xyz="0 0 0" rpy="0 0 -${pi / 2}" />
         <geometry>
           <mesh filename="package://aerial_manipulators/meshes/wp_manipulator/link2.dae"
@@ -40,13 +53,13 @@
     <link name='link3'>
       <inertial>
-        <mass value="0.1" />
-        <origin xyz="0 0 0" rpy="0 0 0"/>
+        <mass value="${mass3}" />
+        <origin xyz="${a3/2} 0 0" rpy="0 0 0"/>
         <inertia
-          ixx="0.01176" ixy="0" ixz="0"
-          iyx="0" iyy="0.01176" iyz="0"
-          izx="0" izy="0" izz="0.0252"/>
+          ixx="${1/2 * mass3 * rad * rad}" ixy="0" ixz="0"
+          iyx="0" iyy="${1/12 * mass3 * (3*rad*rad + a3*a3)}" iyz="0"
+          izx="0" izy="0" izz="${1/12 * mass3 * (3*rad*rad + a3*a3)}"/>
       </inertial>
       <visual>
-        <origin xyz="0 0 0" rpy="${pi / 2} 0 0" />
+        <origin xyz="0 0 0" rpy="0 ${pi / 2} -${pi / 2}" />
         <geometry>
           <mesh filename="package://aerial_manipulators/meshes/wp_manipulator/link3.dae"
@@ -57,13 +70,13 @@
     <link name='link4'>
       <inertial>
-        <mass value="0.1" />
-        <origin xyz="0 0 0" rpy="0 0 0"/>
+        <mass value="${mass4}" />
+        <origin xyz="${a4/2} 0 0" rpy="0 0 0"/>
         <inertia
-          ixx="0.01176" ixy="0" ixz="0"
-          iyx="0" iyy="0.01176" iyz="0"
-          izx="0" izy="0" izz="0.0252"/>
+          ixx="${1/2 * mass4 * rad * rad}" ixy="0" ixz="0"
+          iyx="0" iyy="${1/12 * mass4 * (3*rad*rad + a4*a4)}" iyz="0"
+          izx="0" izy="0" izz="${1/12 * mass4 * (3*rad*rad + a4*a4)}"/>
       </inertial>
       <visual>
-        <origin xyz="0 0 0" rpy="${pi / 2} 0 0" />
+        <origin xyz="0 0 0" rpy="0 ${pi / 2} -${pi / 2}" />
         <geometry>
           <mesh filename="package://aerial_manipulators/meshes/wp_manipulator/link4.dae"
@@ -74,13 +87,13 @@
     <link name='link5'>
       <inertial>
-        <mass value="0.1" />
-        <origin xyz="0 0 0" rpy="0 0 0"/>
+        <mass value="${mass5}" />
+        <origin xyz="${d5/2} 0 0" rpy="0 0 0"/>
         <inertia
-          ixx="0.01176" ixy="0" ixz="0"
-          iyx="0" iyy="0.01176" iyz="0"
-          izx="0" izy="0" izz="0.0252"/>
+          ixx="${1/2 * mass5 * rad * rad}" ixy="0" ixz="0"
+          iyx="0" iyy="${1/12 * mass5 * (3*rad*rad + d5*d5)}" iyz="0"
+          izx="0" izy="0" izz="${1/12 * mass5 * (3*rad*rad + d5*d5)}"/>
       </inertial>
       <visual>
-        <origin xyz="0 0 0" rpy="0 0 0" />
+        <origin xyz="0 0 0" rpy="0 ${pi / 2} 0" />
         <geometry>
           <mesh filename="package://aerial_manipulators/meshes/wp_manipulator/link5.dae"
@@ -92,7 +105,8 @@
       <parent link="world"/>
       <child link="link1"/>
-      <origin xyz="0 0 0" rpy="0 0 0"/>
+      <!-- Adjust Gazebo coordinate system to link1 coordinate system -->
+      <origin xyz="0 0 0" rpy="${pi/2} 0 ${pi}"/>
       <limit upper="3.14" lower="-3.14" effort="10000000" velocity="20"/>
-      <axis xyz="0 1 0" />
+      <axis xyz="0 0 1" />
       <dynamics damping="0.00" friction="0.0"/>
     </joint>
@@ -100,7 +114,7 @@
       <parent link="link1"/>
       <child link="link2"/>
-      <origin xyz="0 0 0" rpy="0 0 0"/>
+      <origin xyz="0 ${a1} 0" rpy="0 0 ${theta1}"/>
       <limit upper="3.14" lower="-3.14" effort="10000000" velocity="20"/>
-      <axis xyz="0 1 0" />
+      <axis xyz="0 0 1" />
       <dynamics damping="0.00" friction="0.0"/>
     </joint>
@@ -108,7 +122,7 @@
       <parent link="link2"/>
       <child link="link3"/>
-      <origin xyz="0 0 0.1365" rpy="0 0 0"/>
+      <origin xyz="${a2} 0 0" rpy="${alpha2} 0 0"/>
       <limit upper="3.14" lower="-3.14" effort="10000000" velocity="20"/>
-      <axis xyz="1 0 0" />
+      <axis xyz="0 0 1" />
       <dynamics damping="0.00" friction="0.0"/>
     </joint>
@@ -116,7 +130,7 @@
       <parent link="link3"/>
       <child link="link4"/>
-      <origin xyz="0 0 0.075511" rpy="0 0 0"/>
+      <origin xyz="${a3} 0 0" rpy="0 0 0"/>
       <limit upper="3.14" lower="-3.14" effort="10000000" velocity="20"/>
-      <axis xyz="1 0 0" />
+      <axis xyz="0 0 1" />
       <dynamics damping="0.00" friction="0.0"/>
     </joint>
@@ -124,7 +138,7 @@
       <parent link="link4"/>
       <child link="link5"/>
-      <origin xyz="0 0 0.072489" rpy="0 0 0"/>
+      <origin xyz="${a4} 0 0" rpy="0 0 0"/>
       <limit upper="3.14" lower="-3.14" effort="10000000" velocity="20"/>
-      <axis xyz="1 0 0" />
+      <axis xyz="0 0 1" />
       <dynamics damping="0.00" friction="0.0"/>
     </joint>

Commit message: Small changes for before Merge

File: urdf/manipulator_base.urdf.xacro (robot description, xacro)
@@ -4,11 +4,11 @@
   params="parent *origin">
     <xacro:property name="a1" value="0.122490"/>
-    <xacro:property name="a2" value="0.136500"/>
+    <xacro:property name="a2" value="0.1365"/>
     <xacro:property name="a3" value="0.075511"/>
     <xacro:property name="a4" value="0.072489"/>
     <xacro:property name="d5" value="0.04526"/>
     <xacro:property name="theta1" value="${pi/2}"/>
-    <xacro:property name="alpha2" value="-${pi/2}"/>
-    <xacro:property name="mass2" value="0.003"/>
+    <xacro:property name="alpha2" value="${-pi/2}"/>
+    <xacro:property name="mass2" value="0.03"/>
     <xacro:property name="mass1" value="${mass2*a1/a2}"/>
     <xacro:property name="mass3" value="${mass2*a3/a2}"/>
@@ -36,5 +36,5 @@
     <link name='link2'>
       <inertial>
-        <mass value="0.03" />
+        <mass value="${mass2}" />
         <origin xyz="${a2/2} 0 0" rpy="0 0 0"/>
         <inertia
@@ -61,5 +61,5 @@
       </inertial>
       <visual>
-        <origin xyz="0 0 0" rpy="0 ${pi / 2} -${pi / 2}" />
+        <origin xyz="0 0 0" rpy="0 ${pi / 2} ${-pi / 2}" />
         <geometry>
           <mesh filename="package://aerial_manipulators/meshes/wp_manipulator/link3.dae"
@@ -102,37 +102,37 @@
       </visual>
     </link>
-    <joint name="link0_to_link1" type="continuous">
+    <joint name="link0_to_link1" type="revolute">
       <parent link="world"/>
       <child link="link1"/>
       <!-- Adjust Gazebo coordinate system to link1 coordinate system -->
       <origin xyz="0 0 0" rpy="${pi/2} 0 ${pi}"/>
-      <limit upper="3.14" lower="-3.14" effort="10000000" velocity="20"/>
+      <limit upper="0" lower="0" effort="10000000" velocity="20"/>
       <axis xyz="0 0 1" />
-      <dynamics damping="0.00" friction="0.0"/>
+      <dynamics damping="0.07" friction="0.01"/>
     </joint>
-    <joint name="link1_to_link2" type="continuous">
+    <joint name="link1_to_link2" type="revolute">
       <parent link="link1"/>
       <child link="link2"/>
       <origin xyz="0 ${a1} 0" rpy="0 0 ${theta1}"/>
-      <limit upper="3.14" lower="-3.14" effort="10000000" velocity="20"/>
+      <limit upper="0" lower="0" effort="10000000" velocity="20"/>
       <axis xyz="0 0 1" />
-      <dynamics damping="0.00" friction="0.0"/>
+      <dynamics damping="0.07" friction="0.01"/>
     </joint>
-    <joint name="link2_to_link3" type="continuous">
+    <joint name="link2_to_link3" type="revolute">
       <parent link="link2"/>
       <child link="link3"/>
       <origin xyz="${a2} 0 0" rpy="${alpha2} 0 0"/>
-      <limit upper="3.14" lower="-3.14" effort="10000000" velocity="20"/>
+      <limit upper="0" lower="0" effort="10000000" velocity="20"/>
       <axis xyz="0 0 1" />
-      <dynamics damping="0.00" friction="0.0"/>
+      <dynamics damping="0.07" friction="0.01"/>
     </joint>
-    <joint name="link3_to_link4" type="continuous">
+    <joint name="link3_to_link4" type="revolute">
       <parent link="link3"/>
       <child link="link4"/>
       <origin xyz="${a3} 0 0" rpy="0 0 0"/>
-      <limit upper="3.14" lower="-3.14" effort="10000000" velocity="20"/>
+      <limit upper="0" lower="0" effort="10000000" velocity="20"/>
       <axis xyz="0 0 1" />
-      <dynamics damping="0.00" friction="0.0"/>
     </joint>
+<!-- <limit upper="1.57" lower="-1.57" effort="10000000" velocity="20"/> -->
     <joint name="link4_to_link5" type="continuous">
       <parent link="link4"/>
@@ -141,6 +141,6 @@
       <limit upper="3.14" lower="-3.14" effort="10000000" velocity="20"/>
       <axis xyz="0 0 1" />
-      <dynamics damping="0.00" friction="0.0"/>
     </joint>
+<!--       <limit upper="2.3" lower="-2.3" effort="10000000" velocity="20"/> -->
   </xacro:macro>
   <!-- We add a <transmission> block for every joint that we wish to actuate. -->

Commit message: Added joint0 parameters

File: urdf/manipulator_base.urdf.xacro (robot description, xacro)
@@ -117,5 +117,5 @@
       <limit upper="0" lower="0" effort="10000000" velocity="20"/>
       <axis xyz="0 0 1" />
-      <dynamics damping="0.07" friction="0.01"/>
+      <dynamics damping="0.07" friction="0.1"/>
     </joint>
     <joint name="link2_to_link3" type="revolute">

Commit message: Added joint limits

File: urdf/manipulator_base.urdf.xacro (robot description, xacro)
@@ -107,5 +107,5 @@
       <!-- Adjust Gazebo coordinate system to link1 coordinate system -->
       <origin xyz="0 0 0" rpy="${pi/2} 0 ${pi}"/>
-      <limit upper="0" lower="0" effort="10000000" velocity="20"/>
+      <limit upper="3.14" lower="-3.14" effort="10000000" velocity="20"/>
       <axis xyz="0 0 1" />
       <dynamics damping="0.07" friction="0.01"/>
@@ -115,5 +115,5 @@
       <child link="link2"/>
       <origin xyz="0 ${a1} 0" rpy="0 0 ${theta1}"/>
-      <limit upper="0" lower="0" effort="10000000" velocity="20"/>
+      <limit upper="3.14" lower="-3.14" effort="10000000" velocity="20"/>
       <axis xyz="0 0 1" />
       <dynamics damping="0.07" friction="0.1"/>
@@ -123,5 +123,5 @@
       <child link="link3"/>
       <origin xyz="${a2} 0 0" rpy="${alpha2} 0 0"/>
-      <limit upper="0" lower="0" effort="10000000" velocity="20"/>
+      <limit upper="3.14" lower="-3.14" effort="10000000" velocity="20"/>
       <axis xyz="0 0 1" />
       <dynamics damping="0.07" friction="0.01"/>
@@ -134,5 +134,4 @@
       <axis xyz="0 0 1" />
     </joint>
-<!-- <limit upper="1.57" lower="-1.57" effort="10000000" velocity="20"/> -->
     <joint name="link4_to_link5" type="continuous">
       <parent link="link4"/>
@@ -142,5 +141,4 @@
       <axis xyz="0 0 1" />
     </joint>
-<!--       <limit upper="2.3" lower="-2.3" effort="10000000" velocity="20"/> -->
   </xacro:macro>
   <!-- We add a <transmission> block for every joint that we wish to actuate. -->

Commit message: Tuned joint4

File: urdf/manipulator_base.urdf.xacro (robot description, xacro)
@@ -107,5 +107,5 @@
       <!-- Adjust Gazebo coordinate system to link1 coordinate system -->
       <origin xyz="0 0 0" rpy="${pi/2} 0 ${pi}"/>
-      <limit upper="3.14" lower="-3.14" effort="10000000" velocity="20"/>
+      <limit upper="0" lower="0" effort="10000000" velocity="20"/>
       <axis xyz="0 0 1" />
       <dynamics damping="0.07" friction="0.01"/>
@@ -115,7 +115,7 @@
       <child link="link2"/>
       <origin xyz="0 ${a1} 0" rpy="0 0 ${theta1}"/>
-      <limit upper="3.14" lower="-3.14" effort="10000000" velocity="20"/>
+      <limit upper="0" lower="0" effort="10000000" velocity="20"/>
       <axis xyz="0 0 1" />
-      <dynamics damping="0.07" friction="0.1"/>
+      <dynamics damping="0.07" friction="0.01"/>
     </joint>
     <joint name="link2_to_link3" type="revolute">
@@ -123,5 +123,5 @@
       <child link="link3"/>
       <origin xyz="${a2} 0 0" rpy="${alpha2} 0 0"/>
-      <limit upper="3.14" lower="-3.14" effort="10000000" velocity="20"/>
+      <limit upper="0" lower="0" effort="10000000" velocity="20"/>
       <axis xyz="0 0 1" />
       <dynamics damping="0.07" friction="0.01"/>
@@ -131,13 +131,15 @@
       <child link="link4"/>
       <origin xyz="${a3} 0 0" rpy="0 0 0"/>
-      <limit upper="0" lower="0" effort="10000000" velocity="20"/>
+      <limit upper="2.355" lower="-2.355" effort="10000000" velocity="20"/>
       <axis xyz="0 0 1" />
+      <dynamics damping="0.07" friction="0.01"/>
     </joint>
-    <joint name="link4_to_link5" type="continuous">
+    <joint name="link4_to_link5" type="revolute">
       <parent link="link4"/>
       <child link="link5"/>
       <origin xyz="${a4} 0 0" rpy="0 0 0"/>
-      <limit upper="3.14" lower="-3.14" effort="10000000" velocity="20"/>
+      <limit upper="2.355" lower="-2.355" effort="10000000" velocity="20"/>
       <axis xyz="0 0 1" />
+      <dynamics damping="0.07" friction="0.01"/>
     </joint>
   </xacro:macro>

Commit message: Reverted tuning changes, added prefilter, set correct joint parameters

File: urdf/manipulator_base.urdf.xacro (robot description, xacro)
@@ -107,7 +107,7 @@
       <!-- Adjust Gazebo coordinate system to link1 coordinate system -->
       <origin xyz="0 0 0" rpy="${pi/2} 0 ${pi}"/>
-      <limit upper="0" lower="0" effort="10000000" velocity="20"/>
+      <limit upper="0" lower="0" effort="1.62" velocity="11.9"/>
       <axis xyz="0 0 1" />
-      <dynamics damping="0.07" friction="0.01"/>
+      <dynamics friction="0.13"/>
     </joint>
     <joint name="link1_to_link2" type="revolute">
@@ -115,7 +115,7 @@
       <child link="link2"/>
       <origin xyz="0 ${a1} 0" rpy="0 0 ${theta1}"/>
-      <limit upper="0" lower="0" effort="10000000" velocity="20"/>
+      <limit upper="0" lower="0" effort="1.62" velocity="11.9"/>
       <axis xyz="0 0 1" />
-      <dynamics damping="0.07" friction="0.01"/>
+      <dynamics friction="0.13"/>
     </joint>
     <joint name="link2_to_link3" type="revolute">
@@ -123,7 +123,7 @@
       <child link="link3"/>
       <origin xyz="${a2} 0 0" rpy="${alpha2} 0 0"/>
-      <limit upper="0" lower="0" effort="10000000" velocity="20"/>
+      <limit upper="0.0" lower="0.0" effort="1.62" velocity="11.9"/>
       <axis xyz="0 0 1" />
-      <dynamics damping="0.07" friction="0.01"/>
+      <dynamics friction="0.13"/>
     </joint>
     <joint name="link3_to_link4" type="revolute">
@@ -131,7 +131,7 @@
       <child link="link4"/>
       <origin xyz="${a3} 0 0" rpy="0 0 0"/>
-      <limit upper="2.355" lower="-2.355" effort="10000000" velocity="20"/>
+      <limit upper="0.0" lower="0.0" effort="1.62" velocity="11.9"/>
       <axis xyz="0 0 1" />
-      <dynamics damping="0.07" friction="0.01"/>
+      <dynamics friction="0.13"/>
     </joint>
     <joint name="link4_to_link5" type="revolute">
@@ -139,7 +139,7 @@
       <child link="link5"/>
       <origin xyz="${a4} 0 0" rpy="0 0 0"/>
-      <limit upper="2.355" lower="-2.355" effort="10000000" velocity="20"/>
+      <limit upper="2.355" lower="-2.355" effort="1.62" velocity="11.9"/>
       <axis xyz="0 0 1" />
-      <dynamics damping="0.07" friction="0.01"/>
+      <dynamics friction="0.13"/>
     </joint>
   </xacro:macro>

Commit message: Joint 5 tuned

File: urdf/manipulator_base.urdf.xacro (robot description, xacro)
@@ -141,5 +141,5 @@
       <limit upper="2.355" lower="-2.355" effort="1.62" velocity="11.9"/>
       <axis xyz="0 0 1" />
-      <dynamics friction="0.13"/>
+      <dynamics friction="0.05"/>
     </joint>
   </xacro:macro>

Commit message: Joint 5 tuned

File: urdf/manipulator_base.urdf.xacro (robot description, xacro)
@@ -131,7 +131,7 @@
       <child link="link4"/>
       <origin xyz="${a3} 0 0" rpy="0 0 0"/>
-      <limit upper="0.0" lower="0.0" effort="1.62" velocity="11.9"/>
+      <limit upper="0.0" lower="0.0" effort="3.1" velocity="11.9"/>
       <axis xyz="0 0 1" />
-      <dynamics friction="0.13"/>
+      <dynamics friction="0.05"/>
     </joint>
     <joint name="link4_to_link5" type="revolute">
@@ -139,5 +139,5 @@
       <child link="link5"/>
       <origin xyz="${a4} 0 0" rpy="0 0 0"/>
-      <limit upper="2.355" lower="-2.355" effort="1.62" velocity="11.9"/>
+      <limit upper="2.355" lower="-2.355" effort="3.1" velocity="11.9"/>
       <axis xyz="0 0 1" />
       <dynamics friction="0.05"/>

Commit message: Set zero friction and damping

File: urdf/manipulator_base.urdf.xacro (robot description, xacro)
@@ -109,5 +109,5 @@
       <limit upper="0" lower="0" effort="1.62" velocity="11.9"/>
       <axis xyz="0 0 1" />
-      <dynamics friction="0.13"/>
+      <dynamics friction="0.0" damping="0.0"/>
     </joint>
     <joint name="link1_to_link2" type="revolute">
@@ -117,5 +117,5 @@
       <limit upper="0" lower="0" effort="1.62" velocity="11.9"/>
       <axis xyz="0 0 1" />
-      <dynamics friction="0.13"/>
+      <dynamics friction="0.0" damping="0.0"/>
     </joint>
     <joint name="link2_to_link3" type="revolute">
@@ -125,5 +125,5 @@
       <limit upper="0.0" lower="0.0" effort="1.62" velocity="11.9"/>
       <axis xyz="0 0 1" />
-      <dynamics friction="0.13"/>
+      <dynamics friction="0.0" damping="0.0"/>
     </joint>
     <joint name="link3_to_link4" type="revolute">
@@ -133,5 +133,5 @@
       <limit upper="0.0" lower="0.0" effort="3.1" velocity="11.9"/>
       <axis xyz="0 0 1" />
-      <dynamics friction="0.05"/>
+      <dynamics friction="0.0" damping="0.0"/>
     </joint>
     <joint name="link4_to_link5" type="revolute">
@@ -139,7 +139,7 @@
       <child link="link5"/>
       <origin xyz="${a4} 0 0" rpy="0 0 0"/>
-      <limit upper="2.355" lower="-2.355" effort="3.1" velocity="11.9"/>
+      <limit upper="2.355" lower="-2.355" effort="6" velocity="11.9"/>
       <axis xyz="0 0 1" />
-      <dynamics friction="0.05"/>
+      <dynamics friction="0.0" damping="0.0"/>
     </joint>
   </xacro:macro>

Commit message: Tuned joint 5 - no friction

File: urdf/manipulator_base.urdf.xacro (robot description, xacro)
@@ -139,5 +139,5 @@
       <child link="link5"/>
       <origin xyz="${a4} 0 0" rpy="0 0 0"/>
-      <limit upper="2.355" lower="-2.355" effort="6" velocity="11.9"/>
+      <limit upper="2.355" lower="-2.355" effort="3.1" velocity="11.9"/>
       <axis xyz="0 0 1" />
       <dynamics friction="0.0" damping="0.0"/>
