Commit message: Tuned position and velocity PIDs

File: urdf/manipulator_base.urdf.xacro (robot description, xacro)
@@ -102,4 +102,19 @@
       </visual>
     </link>
+    <link name="endEffector">
+      <inertial>
+        <mass value="0.00001" />
+        <origin xyz="0 0 0" rpy="0 0 0"/>
+        <inertia
+          ixx="0.00001" ixy="0" ixz="0"
+          iyx="0" iyy="0.00001" iyz="0"
+          izx="0" izy="0" izz="0.00001"/>
+      </inertial>
+      <visual>
+        <geometry>
+          <sphere radius="0.005"/>
+        </geometry>
+      </visual>
+    </link>
     <joint name="link0_to_link1" type="revolute">
       <parent link="world"/>
@@ -107,7 +122,6 @@
       <!-- Adjust Gazebo coordinate system to link1 coordinate system -->
       <origin xyz="0 0 0" rpy="${pi/2} 0 ${pi}"/>
-      <limit upper="0" lower="0" effort="10000000" velocity="20"/>
+      <limit upper="1.57" lower="-1.57" effort="10000000" velocity="20"/>
       <axis xyz="0 0 1" />
-      <dynamics damping="0.07" friction="0.01"/>
     </joint>
     <joint name="link1_to_link2" type="revolute">
@@ -115,7 +129,6 @@
       <child link="link2"/>
       <origin xyz="0 ${a1} 0" rpy="0 0 ${theta1}"/>
-      <limit upper="0" lower="0" effort="10000000" velocity="20"/>
+      <limit upper="2.2" lower="-2.2" effort="10000000" velocity="20"/>
       <axis xyz="0 0 1" />
-      <dynamics damping="0.07" friction="0.01"/>
     </joint>
     <joint name="link2_to_link3" type="revolute">
@@ -123,7 +136,6 @@
       <child link="link3"/>
       <origin xyz="${a2} 0 0" rpy="${alpha2} 0 0"/>
-      <limit upper="0" lower="0" effort="10000000" velocity="20"/>
+      <limit upper="1.57" lower="-1.57" effort="10000000" velocity="20"/>
       <axis xyz="0 0 1" />
-      <dynamics damping="0.07" friction="0.01"/>
     </joint>
     <joint name="link3_to_link4" type="revolute">
@@ -131,16 +143,23 @@
       <child link="link4"/>
       <origin xyz="${a3} 0 0" rpy="0 0 0"/>
+      <limit upper="1.57" lower="-1.57" effort="10000000" velocity="20"/>
+      <axis xyz="0 0 1" />
+    </joint>
+<!-- <limit upper="1.57" lower="-1.57" effort="10000000" velocity="20"/> -->
+    <joint name="link4_to_link5" type="revolute">
+      <parent link="link4"/>
+      <child link="link5"/>
+      <origin xyz="${a4} 0 0" rpy="0 0 0"/>
+      <limit upper="2.3" lower="-2.3" effort="10000000" velocity="20"/>
+      <axis xyz="0 0 1" />
+    </joint>
+<!--       <limit upper="2.3" lower="-2.3" effort="10000000" velocity="20"/> -->
+    <joint name="link5_to_ef" type="revolute">
+      <parent link="link5"/>
+      <child link="endEffector"/>
+      <origin xyz="${d5} 0 0" rpy="${-pi/2} 0 ${-pi/2}"/>
       <limit upper="0" lower="0" effort="10000000" velocity="20"/>
       <axis xyz="0 0 1" />
     </joint>
-<!-- <limit upper="1.57" lower="-1.57" effort="10000000" velocity="20"/> -->
-    <joint name="link4_to_link5" type="continuous">
-      <parent link="link4"/>
-      <child link="link5"/>
-      <origin xyz="${a4} 0 0" rpy="0 0 0"/>
-      <limit upper="3.14" lower="-3.14" effort="10000000" velocity="20"/>
-      <axis xyz="0 0 1" />
-    </joint>
-<!--       <limit upper="2.3" lower="-2.3" effort="10000000" velocity="20"/> -->
   </xacro:macro>
   <!-- We add a <transmission> block for every joint that we wish to actuate. -->

Commit message: Adjusted joint4 effort

File: urdf/manipulator_base.urdf.xacro (robot description, xacro)
@@ -131,5 +131,5 @@
       <child link="link4"/>
       <origin xyz="${a3} 0 0" rpy="0 0 0"/>
-      <limit upper="2" lower="-2" effort="3.1" velocity="11.9"/>
+      <limit upper="2" lower="-2" effort="1.62" velocity="11.9"/>
       <axis xyz="0 0 1" />
       <dynamics friction="0.0" damping="0.0"/>

Commit message: CMake cleanup, configured joint limits

File: urdf/manipulator_base.urdf.xacro (robot description, xacro)
@@ -139,5 +139,5 @@
       <child link="link5"/>
       <origin xyz="${a4} 0 0" rpy="0 0 0"/>
-      <limit upper="1.5" lower="-1.5" effort="1.62" velocity="11.9"/>
+      <limit upper="2" lower="-2" effort="1.62" velocity="11.9"/>
       <axis xyz="0 0 1" />
       <dynamics friction="0.005" damping="0.0"/>

Commit message: created new branch

File: urdf/manipulator_base.urdf.xacro (robot description, xacro)
@@ -1,6 +1,7 @@
 <?xml version="1.0"?>
 <robot xmlns:xacro="http://ros.org/wiki/xacro">
-  <xacro:macro name="cmanip"
+  <xacro:macro name="wp_manipulator"
   params="parent *origin">
+    <xacro:property name="a0" value="0.04526"/>
     <xacro:property name="a1" value="0.122490"/>
     <xacro:property name="a2" value="0.1365"/>
@@ -17,4 +18,21 @@
     <xacro:property name="rad" value="0.03"/>
     <link name="world"></link>
+    <link name='link0'>
+      <inertial>
+        <mass value="${mass5}" />
+        <origin xyz="0 ${a0/2} 0" rpy="0 0 0"/>
+        <inertia
+          ixx="${1/12 * mass5 * (3*rad*rad + a0*a0)}" ixy="0" ixz="0"
+          iyx="0" iyy="${1/2 * mass5 * rad * rad}" iyz="0"
+          izx="0" izy="0" izz="${1/12 * mass5 * (3*rad*rad + a0*a0)}"/>
+      </inertial>
+      <visual>
+        <origin xyz="0 0 0" rpy="${pi / 2} 0 ${pi}" />
+        <geometry>
+          <mesh filename="package://aerial_manipulators/meshes/wp_manipulator/base.dae"
+            scale="1 1 1" />
+        </geometry>
+      </visual>
+    </link>
     <link name='link1'>
       <inertial>
@@ -102,21 +120,12 @@
       </visual>
     </link>
-    <link name="endEffector">
-      <inertial>
-        <mass value="0.00001" />
-        <origin xyz="0 0 0" rpy="0 0 0"/>
-        <inertia
-          ixx="0.00001" ixy="0" ixz="0"
-          iyx="0" iyy="0.00001" iyz="0"
-          izx="0" izy="0" izz="0.00001"/>
-      </inertial>
-      <visual>
-        <geometry>
-          <sphere radius="0.005"/>
-        </geometry>
-      </visual>
-    </link>
-    <joint name="link0_to_link1" type="revolute">
+    <joint name="world_to_link0" type="fixed">
       <parent link="world"/>
+      <child link="link0"/>
+      <!-- Adjust Gazebo coordinate system to link1 coordinate system -->
+      <origin xyz="0 0 ${a0}" rpy="0 0 0"/>
+    </joint>
+    <joint name="link0_to_link1" type="fixed">
+      <parent link="link0"/>
       <child link="link1"/>
       <!-- Adjust Gazebo coordinate system to link1 coordinate system -->
@@ -125,5 +134,5 @@
       <axis xyz="0 0 1" />
     </joint>
-    <joint name="link1_to_link2" type="revolute">
+    <joint name="link1_to_link2" type="fixed">
       <parent link="link1"/>
       <child link="link2"/>
@@ -132,5 +141,5 @@
       <axis xyz="0 0 1" />
     </joint>
-    <joint name="link2_to_link3" type="revolute">
+    <joint name="link2_to_link3" type="fixed">
       <parent link="link2"/>
       <child link="link3"/>
@@ -139,5 +148,5 @@
       <axis xyz="0 0 1" />
     </joint>
-    <joint name="link3_to_link4" type="revolute">
+    <joint name="link3_to_link4" type="fixed">
       <parent link="link3"/>
       <child link="link4"/>
@@ -147,5 +156,5 @@
     </joint>
 <!-- <limit upper="1.57" lower="-1.57" effort="10000000" velocity="20"/> -->
-    <joint name="link4_to_link5" type="revolute">
+    <joint name="link4_to_link5" type="fixed">
       <parent link="link4"/>
       <child link="link5"/>
@@ -155,11 +164,4 @@
     </joint>
 <!--       <limit upper="2.3" lower="-2.3" effort="10000000" velocity="20"/> -->
-    <joint name="link5_to_ef" type="revolute">
-      <parent link="link5"/>
-      <child link="endEffector"/>
-      <origin xyz="${d5} 0 0" rpy="${-pi/2} 0 ${-pi/2}"/>
-      <limit upper="0" lower="0" effort="10000000" velocity="20"/>
-      <axis xyz="0 0 1" />
-    </joint>
   </xacro:macro>
   <!-- We add a <transmission> block for every joint that we wish to actuate. -->

File: urdf/wp_manipulator.base.urdf.xacro (robot description, xacro)
@@ -1,9 +1,9 @@
 <?xml version="1.0"?>
-<robot name="cmanip" xmlns:xacro="http://ros.org/wiki/xacro">
+<robot name="wp_manipulator" xmlns:xacro="http://ros.org/wiki/xacro">
   <xacro:include filename="$(find aerial_manipulators)/urdf/manipulator_base.urdf.xacro" />
-  <xacro:cmanip
+  <xacro:wp_manipulator
     parent="world">
     <origin xyz="0 0 0" rpy="0 0 0"/>
-  </xacro:cmanip>
+  </xacro:wp_manipulator>
   <xacro:transmisija
     trans_number="1"

File: urdf/wp_manipulator.gazebo.xacro (robot description, xacro)
@@ -1,4 +1,4 @@
 <?xml version="1.0"?>
-<robot name="cmanip" xmlns:xacro="http://ros.org/wiki/xacro">
+<robot name="wp_manipulator" xmlns:xacro="http://ros.org/wiki/xacro">
   <!--
   It seems that the xacro:property does not allow to use substitution args. Therefore, instead xacro parameter ${namespace}, subsitution argument is used $(arg name). This is
@@ -8,9 +8,9 @@
   <xacro:property name="bag_file" value="cmanip.bag" />
   <!-- Instantiate cmanip "mechanics" -->
-  <xacro:include filename="$(find aerial_manipulators)/urdf/cmanip.base.urdf.xacro" />
-  <gazebo>
+  <xacro:include filename="$(find aerial_manipulators)/urdf/wp_manipulator.base.urdf.xacro" />
+  <!--gazebo>
     <plugin name="gazebo_ros_control" filename="libgazebo_ros_control.so">
       <robotNamespace>/cmanip</robotNamespace>
     </plugin>
-  </gazebo>
+  </gazebo-->
 </robot>

Commit message: Removed Gravity From Force Sensor

File: urdf/manipulator_base.urdf.xacro (robot description, xacro)
@@ -98,15 +98,24 @@
       <inertial>
         <mass value="0.00001" />
-        <origin xyz="0 0 0" rpy="0 0 0"/>
+        <origin rpy="0 0 0" xyz="0 0 -0.02998408"/>
         <inertia
-          ixx="0.00001" ixy="0" ixz="0"
-          iyx="0" iyy="0.00001" iyz="0"
-          izx="0" izy="0" izz="0.00001"/>
-      </inertial>
-      <visual>
-        <geometry>
-          <sphere radius="0.005"/>
-        </geometry>
-      </visual>
+          ixx="0.000001" ixy="0" ixz="0.0"
+          iyx="0" iyy="0.000001" iyz="0"
+          izx="0.0" izy="0" izz="0.000001"/>
+      </inertial>
+    <visual>
+      <origin xyz="-0.001903 -0.001661 -0.005153" rpy="${-pi/2} 0 ${-pi/2}" />
+      <geometry>
+        <mesh filename="package://aerial_manipulators/meshes/wp_manipulator/forcesensor_mount_top.dae"
+          scale="0.1 0.1 0.1" />
+      </geometry>
+    </visual>
+    <collision name='collision'>
+      <origin xyz="-0.001903 -0.001661 -0.005153" rpy="${-pi/2} 0 ${-pi/2}"/>
+      <geometry>
+        <mesh filename="package://aerial_manipulators/meshes/wp_manipulator/forcesensor_mount_top.dae"
+          scale="0.1 0.1 0.1" />
+      </geometry>
+    </collision>
     </link>
 -->
@@ -154,5 +163,5 @@
       <parent link="link5"/>
       <child link="endEffector"/>
-      <origin xyz="${d5} 0 0" rpy="${-pi/2} 0 ${-pi/2}"/>
+      <origin xyz="${d5} 0 0" rpy="0 0 0"/>
       <limit upper="0" lower="0" effort="10000000" velocity="20"/>
       <axis xyz="0 0 1" />
